File: Steuereinheit.kicad_sch (KiCad schematic)
At the start: 58 parts, among them J1 Tueroeffnunfen, J10 Fadenfoul, J11 Netzteil, J12 Serienplan, J13 Serienplan 2, J14 Muenzeinheit 2, J15 I2C-Bus, J16 Kodierg., J17 TTL-Ein-/Ausgaenge, J18 RS485 Aus, J19 RS485 Ein, J2 PSG In/OUT, J20 Serielle-S., J21 Tuerschalter, J3 Lautsprecher, J4 DIN41612_03x10_ABC, J5 DIN41612_03x10_ABC, J6 Service, J7 Maschine, J8 Muenzeinheit, J9 Akzeptor, U1 74LS573, U10 74HC245, U11 SG-531, U12 74AHCT125, U13 TL7705A, U14 L4974A, U15 68C681, U16 74LS32, U17 74HC138, U18 TC428, U19 SN75176AP, U2 TS271, U20 SN75176AP, U21 LTV-827, U3 74HC02, U4 LM317L_TO92, U5 40374, U6 74LS393, U7 74LS195, U8 AD7224KN, U9 YM2149

Commit message: leiterbahnen
Connections:
- net at U6.2 (MR): now also U6.12 (MR)
- net at U20.6 (A): now also J19.1 (Pin_1)
- net at U20.7 (B): now also J19.2 (Pin_2)
- net at J18.1 (Pin_1): now also U19.6 (A)
- net at J18.2 (Pin_2): now also U19.7 (B)
Other:
- moved on the sheet: J18, J19, U20
Changed lines of the file:
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@@
 	(wire
 		(pts
+			(xy 299.72 261.62) (xy 297.18 261.62)
+		)
+		(stroke
+			(width 0)
+			(type default)
+		)
+	)
+	(wire
+		(pts
 			(xy 176.53 361.95) (xy 176.53 363.22)
 		)
@@
 	(wire
 		(pts
+			(xy 71.12 132.08) (xy 71.12 109.22)
+		)
+		(stroke
+			(width 0)
+			(type default)
+		)
+	)
+	(wire
+		(pts
 			(xy 93.98 254) (xy 86.36 254)
 		)
@@
 	(wire
 		(pts
+			(xy 76.2 132.08) (xy 71.12 132.08)
+		)
+		(stroke
+			(width 0)
+			(type default)
+		)
+	)
+	(wire
+		(pts
+			(xy 299.72 264.16) (xy 297.18 264.16)
+		)
+		(stroke
+			(width 0)
+			(type default)
+		)
+	)
+	(wire
+		(pts
+			(xy 71.12 109.22) (xy 76.2 109.22)
+		)
+		(stroke
+			(width 0)
+			(type default)
+		)
+	)
+	(wire
+		(pts
 			(xy 176.53 363.22) (xy 176.53 364.49)
 		)
@@
 	(wire
 		(pts
+			(xy 299.72 299.72) (xy 297.18 299.72)
+		)
+		(stroke
+			(width 0)
+			(type default)
+		)
+	)
+	(wire
+		(pts
 			(xy 86.36 254) (xy 86.36 261.62)
 		)
@@
 	(wire
 		(pts
+			(xy 299.72 302.26) (xy 297.18 302.26)
+		)
+		(stroke
+			(width 0)
+			(type default)
+		)
+	)
+	(wire
+		(pts
 			(xy 176.53 367.03) (xy 176.53 368.3)
 		)
@@
 	(symbol
 		(lib_id "Interface_UART:SN75176AP")
-		(at 313.69 260.35 0)
+		(at 289.56 297.18 0)
 		(unit 1)
 		(exclude_from_sim no)
@@
 		(fields_autoplaced yes)
 		(property "Reference" "U20"
-			(at 315.8333 247.65 0)
+			(at 291.7033 284.48 0)
 			(effects
 				(font
@@
 		)
 		(property "Value" "SN75176AP"
-			(at 315.8333 250.19 0)
+			(at 291.7033 287.02 0)
 			(effects
 				(font
@@
 		)
 		(property "Footprint" "Package_DIP:DIP-8_W7.62mm"
-			(at 313.69 273.05 0)
+			(at 289.56 309.88 0)
 			(effects
 				(font
@@
 		)
 		(property "Datasheet" "http://www.ti.com/lit/ds/symlink/sn75176a.pdf"
-			(at 354.33 265.43 0)
+			(at 330.2 302.26 0)
 			(effects
 				(font
@@
 		)
 		(property "Description" "Differential RS-422/RS-485 bus transceiver, DIP-8"
-			(at 313.69 260.35 0)
+			(at 289.56 297.18 0)
 			(effects
 				(font
@@
 	(symbol
 		(lib_id "power:+5V")
-		(at 313.69 250.19 0)
+		(at 289.56 287.02 0)
 		(unit 1)
 		(exclude_from_sim no)
@@
 		(fields_autoplaced yes)
 		(property "Reference" "#PWR045"
-			(at 313.69 254 0)
+			(at 289.56 290.83 0)
 			(effects
 				(font
@@
 		)
 		(property "Value" "+5V"
-			(at 313.69 245.11 0)
+			(at 289.56 281.94 0)
 			(effects
 				(font
@@
 		)
 		(property "Footprint" ""
-			(at 313.69 250.19 0)
+			(at 289.56 287.02 0)
 			(effects
 				(font
@@
 		)
 		(property "Datasheet" ""
-			(at 313.69 250.19 0)
+			(at 289.56 287.02 0)
 			(effects
 				(font
@@
 		)
 		(property "Description" "Power symbol creates a global label with name \"+5V\""
-			(at 313.69 250.19 0)
+			(at 289.56 287.02 0)
 			(effects
 				(font
@@
 	(symbol
 		(lib_id "Connector_Generic:Conn_01x02")
-		(at 278.13 367.03 0)
+		(at 304.8 264.16 0)
+		(mirror x)
 		(unit 1)
 		(exclude_from_sim no)
@@
 		(on_board yes)
 		(dnp no)
-		(fields_autoplaced yes)
 		(property "Reference" "J18"
-			(at 280.67 367.0299 0)
+			(at 307.34 264.1601 0)
 			(effects
 				(font
@@
 		)
 		(property "Value" "RS485 Aus"
-			(at 280.67 369.5699 0)
+			(at 307.34 261.6201 0)
 			(effects
 				(font
@@
 		)
 		(property "Footprint" "Connector_PinHeader_2.54mm:PinHeader_1x02_P2.54mm_Vertical"
-			(at 278.13 367.03 0)
+			(at 304.8 264.16 0)
 			(effects
 				(font
@@
 		)
 		(property "Datasheet" "~"
-			(at 278.13 367.03 0)
+			(at 304.8 264.16 0)
 			(effects
 				(font
@@
 		)
 		(property "Description" "Generic connector, single row, 01x02, script generated (kicad-library-utils/schlib/autogen/connector/)"
-			(at 278.13 367.03 0)
+			(at 304.8 264.16 0)
 			(effects
 				(font
@@
 	(symbol
 		(lib_id "Connector_Generic:Conn_01x02")
-		(at 278.13 379.73 0)
+		(at 304.8 302.26 0)
+		(mirror x)
 		(unit 1)
 		(exclude_from_sim no)
@@
 		(on_board yes)
 		(dnp no)
-		(fields_autoplaced yes)
 		(property "Reference" "J19"
-			(at 280.67 379.7299 0)
+			(at 307.34 302.2601 0)
 			(effects
 				(font
@@
 		)
 		(property "Value" "RS485 Ein"
-			(at 280.67 382.2699 0)
+			(at 307.34 299.7201 0)
 			(effects
 				(font
@@
 		)
 		(property "Footprint" "Connector_PinHeader_2.54mm:PinHeader_1x02_P2.54mm_Vertical"
-			(at 278.13 379.73 0)
+			(at 304.8 302.26 0)
 			(effects
 				(font
@@
 		)
 		(property "Datasheet" "~"
-			(at 278.13 379.73 0)
+			(at 304.8 302.26 0)
 			(effects
 				(font
@@
 		)
 		(property "Description" "Generic connector, single row, 01x02, script generated (kicad-library-utils/schlib/autogen/connector/)"
-			(at 278.13 379.73 0)
+			(at 304.8 302.26 0)
 			(effects
 				(font
@@
 	(symbol
 		(lib_id "power:GND")
-		(at 313.69 270.51 0)
+		(at 289.56 307.34 0)
 		(unit 1)
 		(exclude_from_sim no)
@@
 		(fields_autoplaced yes)
 		(property "Reference" "#PWR015"
-			(at 313.69 276.86 0)
+			(at 289.56 313.69 0)
 			(effects
 				(font
@@
 		)
 		(property "Value" "GND"
-			(at 313.69 275.59 0)
+			(at 289.56 312.42 0)
 			(effects
 				(font
@@
 		)
 		(property "Footprint" ""
-			(at 313.69 270.51 0)
+			(at 289.56 307.34 0)
 			(effects
 				(font
@@
 		)
 		(property "Datasheet" ""
-			(at 313.69 270.51 0)
+			(at 289.56 307.34 0)
 			(effects
 				(font
@@
 		)
 		(property "Description" "Power symbol creates a global label with name \"GND\" , ground"
-			(at 313.69 270.51 0)
+			(at 289.56 307.34 0)
 			(effects
 				(font

Commit message: widers
Parts:
- added C1, C13, C2, C21, C3, C4, C5, C6, C7, C8: 100n, Capacitor_THT:C_Axial_L3.8mm_D2.6mm_P7.50mm_Horizontal, symbol Device:C
- added D4, D5: SD103, Diode_THT:D_DO-35_SOD27_P7.62mm_Horizontal, symbol Device:D_Schottky
- added R10: 15k, Resistor_THT:R_Axial_DIN0207_L6.3mm_D2.5mm_P10.16mm_Horizontal, symbol Device:R
- added R11, R119, R12, R13, R14, R15, R17, R20, R22, R23, R9: 1k, Resistor_THT:R_Axial_DIN0207_L6.3mm_D2.5mm_P10.16mm_Horizontal, symbol Device:R
- added R16, R24, R8: 10k, Resistor_THT:R_Axial_DIN0207_L6.3mm_D2.5mm_P10.16mm_Horizontal, symbol Device:R
- added R18, R19: 100, Resistor_THT:R_Axial_DIN0207_L6.3mm_D2.5mm_P10.16mm_Horizontal, symbol Device:R
- added R21, R27, R30, R31, R32: 47, Resistor_THT:R_Axial_DIN0207_L6.3mm_D2.5mm_P10.16mm_Horizontal, symbol Device:R
- added R25, R26, R28, R29: 470, Resistor_THT:R_Axial_DIN0207_L6.3mm_D2.5mm_P10.16mm_Horizontal, symbol Device:R
Connections:
- net +5V: no longer U8.1 (VSS)
- net GND: now also C13.2, C21.2
- net at J6.3 (Pin_3): now also R30.2
- net at J6.4 (Pin_4): now also R31.2
- net at J6.5 (Pin_5): now also R28.1
- net at J8.5 (Pin_5): now also R29.1
- net at U13.3 (CT): now also U13.5 (~{RESET})
- net at U16.12: now also D5.1 (K)
- new net: C6.2, R10.2
- new net: C5.1, R11.2, R9.2
- new net: C5.2, R8.2
Other:
- moved on the sheet: J8, U16D

Commit message: widerstand
Parts:
- added C10, C33: 10u 25V, Capacitor_THT:CP_Radial_Tantal_D4.5mm_P2.50mm, symbol Device:C_Polarized
- added C11, C43, C9: 220uF 50V, Capacitor_THT:CP_Radial_D8.0mm_P5.00mm, symbol Device:C_Polarized
- added C15, C30, C36, C37, C38: 100n, Capacitor_THT:C_Axial_L3.8mm_D2.6mm_P7.50mm_Horizontal, symbol Device:C
- added C17, C18, C24, C25: 2u2 25V, Capacitor_THT:CP_Radial_Tantal_D4.5mm_P2.50mm, symbol Device:C_Polarized
- added C20: 4n7, Capacitor_THT:C_Rect_L9.0mm_W2.5mm_P7.50mm_MKT, symbol Device:C
- added C28: 33p, Capacitor_THT:C_Disc_D3.0mm_W1.6mm_P2.50mm, symbol Device:C
- added C29: 22n, Capacitor_THT:C_Rect_L7.0mm_W2.0mm_P5.00mm, symbol Device:C
- added D15, D3: SD103, Diode_THT:D_DO-35_SOD27_P7.62mm_Horizontal, symbol Device:D_Schottky
- added D7: 1N5908, Diode_THT:D_DO-201AE_P15.24mm_Horizontal, symbol Diode:1N5908
- added L1: 100uH 4A, Inductor_THT:L_Toroid_Vertical_L24.6mm_W15.5mm_P11.44mm_Pulse_KM-4, symbol Device:L
- added R118: 22, Resistor_THT:R_Axial_DIN0207_L6.3mm_D2.5mm_P10.16mm_Horizontal, symbol Device:R
- added R44, R68, R74: 22k, Resistor_THT:R_Axial_DIN0207_L6.3mm_D2.5mm_P10.16mm_Horizontal, symbol Device:R
- added R45, R71, R91: 100, Resistor_THT:R_Axial_DIN0207_L6.3mm_D2.5mm_P10.16mm_Horizontal, symbol Device:R
- added R46, R47, R48, R49, R50, R51, R52, R53, R54, R55, R77, R78, R79, R81, R82, R83, R84, R86, R87, R88: 47, Resistor_THT:R_Axial_DIN0207_L6.3mm_D2.5mm_P10.16mm_Horizontal, symbol Device:R
- added R69: 15k, Resistor_THT:R_Axial_DIN0207_L6.3mm_D2.5mm_P10.16mm_Horizontal, symbol Device:R
- added R70: 10k, Resistor_THT:R_Axial_DIN0207_L6.3mm_D2.5mm_P10.16mm_Horizontal, symbol Device:R
- added R72, R73, R76: 1k, Resistor_THT:R_Axial_DIN0207_L6.3mm_D2.5mm_P10.16mm_Horizontal, symbol Device:R
- added R75: 4,7k, Resistor_THT:R_Axial_DIN0207_L6.3mm_D2.5mm_P10.16mm_Horizontal, symbol Device:R
- added R80, R85, R89, R90: 470, Resistor_THT:R_Axial_DIN0207_L6.3mm_D2.5mm_P10.16mm_Horizontal, symbol Device:R
- J1: value Tueroeffnunfen -> Tueroeffnungen
- U4: footprint Package_TO_SOT_THT:TO-92_Inline -> Package_TO_SOT_THT:TO-92_Wide
Connections:
- net +12V: now also J9.1 (Pin_1); no longer J11.2 (Pin_2)
- net +24V: now also U14.11 (VREF), C30.1, C9.1, R69.1
- net +5V: now also C13.1, C21.1, C7.2, C8.1, J1.6 (Pin_6), J13.7 (Pin_7), J14.7 (Pin_7), J15.1 (Pin_1), J17.9 (Pin_9), J4.a1 (Pin_a1), J4.a7 (Pin_a7), J4.b1 (Pin_b1), J5.a1 (Pin_a1), J5.a7 (Pin_a7), J5.b1 (Pin_b1), J5.c1 (Pin_c1), J6.1 (Pin_1), J7.7 (Pin_7), J8.7 (Pin_7), R19.2, R20.2, R21.1, R5.2, U9.25 (A8), C33.1, C36.1, C37.1, C38.1, D7.1 (A1), R45.1, R75.2; no longer U14.19 (VCC)
- net GND: now also C3.2, C4.1, C7.1, C8.2, D1.2 (A), D2.1 (K), J5.a10 (Pin_a10), J5.a4 (Pin_a4), J5.b10 (Pin_b10), J5.c10 (Pin_c10), R18.2, R29.2, R9.1, U14.15 (P-UVLO), U14.16 (SYNC), U14.5 (CA-OUT), U14.6 (LFF), U20.4 (D), C10.2, C11.2, C17.2, C18.2, C24.2, C25.2, C28.2, C30.2, C33.2, C36.2, C37.2, C38.2, C43.2, C9.2, D7.2 (A2), R44.1, R55.1, R68.1, R70.1, R72.1, R80.1, R85.1, R89.2, R90.2
- net at J9.2 (Pin_2): now also R71.2
- net at R10.1: now also R8.1
- net at R19.1: now also U7.15 (Q0)
- net at U2.3 (+): now also C3.1
- net at R23.2: now also J1.5 (Pin_5)
- net at J2.1 (Pin_1): now also R25.1
- net at J2.2 (Pin_2): now also R26.1
- net at J2.4 (Pin_4): now also R27.1
- net at R6.1: now also C15.1
- net at J3.6 (Pin_6): now also R15.2
- net at U3.1: now also U9.27 (BDIR)
- net at J1.3 (Pin_3): now also R22.2
- net at J1.4 (Pin_4): now also R24.1
Other:
- moved on the sheet: C3, C4, C6, C7, C8, J2, J3, J9, R10, R15, R19, R22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

Commit message: serial
Connections:
- net at J20.1 (Pin_1): now also U21.1
- net at U19.1 (R): now also U12.6
Other:
- moved on the sheet: J18, U12B, U19, U21A
Changed lines of the file:
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@@
 	(wire
 		(pts
-			(xy 299.72 261.62) (xy 297.18 261.62)
+			(xy 356.87 214.63) (xy 354.33 214.63)
 		)
 		(stroke
@@
 	(wire
 		(pts
-			(xy 299.72 264.16) (xy 297.18 264.16)
+			(xy 356.87 217.17) (xy 354.33 217.17)
 		)
 		(stroke
@@
 	(wire
 		(pts
+			(xy 297.18 354.33) (xy 290.83 354.33)
+		)
+		(stroke
+			(width 0)
+			(type default)
+		)
+	)
+	(wire
+		(pts
 			(xy 81.28 48.26) (xy 86.36 48.26)
 		)
@@
 	(wire
 		(pts
+			(xy 290.83 354.33) (xy 290.83 369.57)
+		)
+		(stroke
+			(width 0)
+			(type default)
+		)
+	)
+	(wire
+		(pts
 			(xy 124.46 411.48) (xy 132.08 411.48)
 		)
@@
 	(wire
 		(pts
+			(xy 290.83 369.57) (xy 297.18 369.57)
+		)
+		(stroke
+			(width 0)
+			(type default)
+		)
+	)
+	(wire
+		(pts
 			(xy 176.53 367.03) (xy 176.53 368.3)
 		)
@@
 	(symbol
 		(lib_id "power:+5V")
-		(at 289.56 248.92 0)
+		(at 346.71 201.93 0)
 		(unit 1)
 		(exclude_from_sim no)
@@
 		(fields_autoplaced yes)
 		(property "Reference" "#PWR044"
-			(at 289.56 252.73 0)
+			(at 346.71 205.74 0)
 			(effects
 				(font
@@
 		)
 		(property "Value" "+5V"
-			(at 289.56 243.84 0)
+			(at 346.71 196.85 0)
 			(effects
 				(font
@@
 		)
 		(property "Footprint" ""
-			(at 289.56 248.92 0)
+			(at 346.71 201.93 0)
 			(effects
 				(font
@@
 		)
 		(property "Datasheet" ""
-			(at 289.56 248.92 0)
+			(at 346.71 201.93 0)
 			(effects
 				(font
@@
 		)
 		(property "Description" "Power symbol creates a global label with name \"+5V\""
-			(at 289.56 248.92 0)
+			(at 346.71 201.93 0)
 			(effects
 				(font
@@
 	(symbol
 		(lib_id "Connector_Generic:Conn_01x02")
-		(at 304.8 264.16 0)
+		(at 361.95 217.17 0)
 		(mirror x)
 		(unit 1)
@@
 		(dnp no)
 		(property "Reference" "J18"
-			(at 307.34 264.1601 0)
+			(at 364.49 217.1701 0)
 			(effects
 				(font
@@
 		)
 		(property "Value" "RS485 Aus"
-			(at 307.34 261.6201 0)
+			(at 364.49 214.6301 0)
 			(effects
 				(font
@@
 		)
 		(property "Footprint" "Connector_PinHeader_2.54mm:PinHeader_1x02_P2.54mm_Vertical"
-			(at 304.8 264.16 0)
+			(at 361.95 217.17 0)
 			(effects
 				(font
@@
 		)
 		(property "Datasheet" "~"
-			(at 304.8 264.16 0)
+			(at 361.95 217.17 0)
 			(effects
 				(font
@@
 		)
 		(property "Description" "Generic connector, single row, 01x02, script generated (kicad-library-utils/schlib/autogen/connector/)"
-			(at 304.8 264.16 0)
+			(at 361.95 217.17 0)
 			(effects
 				(font
@@
 	(symbol
 		(lib_id "Interface_UART:SN75176AP")
-		(at 289.56 259.08 0)
+		(at 346.71 212.09 0)
 		(unit 1)
 		(exclude_from_sim no)
@@
 		(fields_autoplaced yes)
 		(property "Reference" "U19"
-			(at 291.7033 246.38 0)
+			(at 348.8533 199.39 0)
 			(effects
 				(font
@@
 		)
 		(property "Value" "SN75176AP"
-			(at 291.7033 248.92 0)
+			(at 348.8533 201.93 0)
 			(effects
 				(font
@@
 		)
 		(property "Footprint" "Package_DIP:DIP-8_W7.62mm"
-			(at 289.56 271.78 0)
+			(at 346.71 224.79 0)
 			(effects
 				(font
@@
 		)
 		(property "Datasheet" "http://www.ti.com/lit/ds/symlink/sn75176a.pdf"
-			(at 330.2 264.16 0)
+			(at 387.35 217.17 0)
 			(effects
 				(font
@@
 		)
 		(property "Description" "Differential RS-422/RS-485 bus transceiver, DIP-8"
-			(at 289.56 259.08 0)
+			(at 346.71 212.09 0)
 			(effects
 				(font
@@
 	(symbol
 		(lib_id "Isolator:LTV-827")
-		(at 342.9 247.65 0)
+		(at 304.8 356.87 0)
 		(unit 1)
 		(exclude_from_sim no)
@@
 		(fields_autoplaced yes)
 		(property "Reference" "U21"
-			(at 342.9 238.76 0)
+			(at 304.8 347.98 0)
 			(effects
 				(font
@@
 		)
 		(property "Value" "LTV-827"
-			(at 342.9 241.3 0)
+			(at 304.8 350.52 0)
 			(effects
 				(font
@@
 		)
 		(property "Footprint" "Package_DIP:DIP-8_W7.62mm"
-			(at 337.82 252.73 0)
+			(at 299.72 361.95 0)
 			(effects
 				(font
@@
 		)
 		(property "Datasheet" "http://optoelectronics.liteon.com/upload/download/DS-70-96-0016/LTV-8X7%20series%20201610%20.pdf"
-			(at 342.9 247.65 0)
+			(at 304.8 356.87 0)
 			(effects
 				(font
@@
 		)
 		(property "Description" "Dual DC Optocoupler, Vce 35V, CTR 50%, DIP-8"
-			(at 342.9 247.65 0)
+			(at 304.8 356.87 0)
 			(effects
 				(font
@@
 	(symbol
 		(lib_id "74xx:74AHCT125")
-		(at 252.73 186.69 0)
+		(at 331.47 217.17 0)
 		(unit 2)
 		(exclude_from_sim no)
@@
 		(fields_autoplaced yes)
 		(property "Reference" "U12"
-			(at 252.73 177.8 0)
+			(at 331.47 208.28 0)
 			(effects
 				(font
@@
 		)
 		(property "Value" "74AHCT125"
-			(at 252.73 180.34 0)
+			(at 331.47 210.82 0)
 			(effects
 				(font
@@
 		)
 		(property "Footprint" "Package_DIP:DIP-14_W7.62mm"
-			(at 252.73 186.69 0)
+			(at 331.47 217.17 0)
 			(effects
 				(font
@@
 		)
 		(property "Datasheet" "https://www.ti.com/lit/ds/symlink/sn74ahct125.pdf"
-			(at 252.73 186.69 0)
+			(at 331.47 217.17 0)
 			(effects
 				(font
@@
 		)
 		(property "Description" "Quadruple Bus Buffer Gates With 3-State Outputs"
-			(at 252.73 186.69 0)
+			(at 331.47 217.17 0)
 			(effects
 				(font
@@
 	(symbol
 		(lib_id "power:GND")
-		(at 289.56 269.24 0)
+		(at 346.71 222.25 0)
 		(unit 1)
 		(exclude_from_sim no)
@@
 		(fields_autoplaced yes)
 		(property "Reference" "#PWR014"
-			(at 289.56 275.59 0)
+			(at 346.71 228.6 0)
 			(effects
 				(font
@@
 		)
 		(property "Value" "GND"
-			(at 289.56 274.32 0)
+			(at 346.71 227.33 0)
 			(effects
 				(font
@@
 		)
 		(property "Footprint" ""
-			(at 289.56 269.24 0)
+			(at 346.71 222.25 0)
 			(effects
 				(font
@@
 		)
 		(property "Datasheet" ""
-			(at 289.56 269.24 0)
+			(at 346.71 222.25 0)
 			(effects
 				(font
@@
 		)
 		(property "Description" "Power symbol creates a global label with name \"GND\" , ground"
-			(at 289.56 269.24 0)
+			(at 346.71 222.25 0)
 			(effects
 				(font

Commit message: alle bauteile
Parts:
- removed U14: L4974A, Package_DIP:DIP-20_W7.62mm, symbol Regulator_Controller:L4981A
- added C12, C14, C16, C22, C23, C26, C31, C32, C39, C40: 100n, Capacitor_THT:C_Axial_L3.8mm_D2.6mm_P7.50mm_Horizontal, symbol Device:C
- added C20: 4n7, Capacitor_THT:C_Rect_L7.0mm_W2.0mm_P5.00mm, symbol Device:C
- added C35, C41, C9: 10u 25V, Capacitor_THT:CP_Radial_Tantal_D4.5mm_P2.50mm, symbol Device:C_Polarized
- added C42: 470n, Capacitor_THT:C_Rect_L9.0mm_W2.5mm_P7.50mm_MKT, symbol Device:C
- added D10, D11, D12, D13, D14, D6, D8, D9: SD103, Diode_THT:D_DO-35_SOD27_P7.62mm_Horizontal, symbol Device:D_Schottky
- added Q1, Q2: BSS100, Package_TO:TO-92, symbol Transistor_FET:BSS123
- added Q10, Q11, Q12, Q4, Q5, Q6, Q7, Q8: BC337, Package_TO:TO-92, symbol Transistor_BJT:BC337
- added Q3, Q9: BC327, Package_TO:TO-92, symbol Transistor_BJT:BC327
- added R100, R101, R33, R37, R38, R92, R94, R97: 100, Resistor_THT:R_Axial_DIN0207_L6.3mm_D2.5mm_P10.16mm_Horizontal, symbol Device:R
- added R102, R104, R107, R116, R117, R59, R93, R96, R98: 1k, Resistor_THT:R_Axial_DIN0207_L6.3mm_D2.5mm_P10.16mm_Horizontal, symbol Device:R
- added R103, R109, R110, R111, R112, R113, R56, R57, R58, R63: 10k, Resistor_THT:R_Axial_DIN0207_L6.3mm_D2.5mm_P10.16mm_Horizontal, symbol Device:R
- added R105, R106, R114, R36, R62, R64, R67: 470, Resistor_THT:R_Axial_DIN0207_L6.3mm_D2.5mm_P10.16mm_Horizontal, symbol Device:R
- added R108, R65, R95, R99: 4,7k, Resistor_THT:R_Axial_DIN0207_L6.3mm_D2.5mm_P10.16mm_Horizontal, symbol Device:R
- added R115, R39, R40, R41, R42, R43: 47, Resistor_THT:R_Axial_DIN0207_L6.3mm_D2.5mm_P10.16mm_Horizontal, symbol Device:R
- added R34: 210, Resistor_THT:R_Axial_DIN0207_L6.3mm_D2.5mm_P10.16mm_Horizontal, symbol Device:R
- added R35: 499, Resistor_THT:R_Axial_DIN0207_L6.3mm_D2.5mm_P10.16mm_Horizontal, symbol Device:R
- added R60, R61, R66: 220, Resistor_THT:R_Axial_DIN0207_L6.3mm_D2.5mm_P10.16mm_Horizontal, symbol Device:R
- added U14: ~, Package_DIP:DIP-20_W7.62mm, symbol Power_ST:L4974A
- C19: renamed from C20; value 4n7 -> 470n
- U4: footprint Package_TO_SOT_THT:TO-92_Wide -> Package_TO:TO-92; now not fitted
- U8: now not fitted
- renumbered C9 to C34
Connections:
- net +24V: now also U14.11 (Vi)
- net +5V: now also U13.7 (SENSE), C12.1, C14.1, C16.1, C31.1, C35.1, C39.1, C40.1, C41.1, C9.1, D10.1 (K), R36.2
- net GND: now also C12.2, C14.2, C16.2, C20.1, C22.2, C23.2, C26.2, C31.2, C35.2, C39.2, C40.2, C41.2, C42.1, C9.2, D10.2 (A), Q1.3 (D), Q10.3 (E), Q2.3 (D), Q3.1 (C), Q4.3 (E), Q7.3 (E), Q9.1 (C), R103.2, R35.1, R57.1, R58.2, U14.15 (GND), U14.16 (GND), U14.5 (GND), U14.6 (GND)
- net at U6.12 (MR), U6.2 (MR): now also R18.1
- net at L1.1: now also C19.2, D1.1 (K), U14.20 (Output)
- net at L1.2: now also C1.1, C11.1, C43.1
- net at R20.1: now also U12.1
- net at D4.2 (A): now also D5.2 (A)
- net at D17.1 (K): now also Q3.3 (E)
- net at D17.2 (A): now also R92.1
- net at D16.1 (K): now also Q9.3 (E)
- net at J19.2 (Pin_2), U20.7 (B): now also R56.2
- net at U17.6 (E2): now also U7.7 (P3)
- net at J5.a6 (Pin_a6): now also R14.2
- net at R15.1: now also U12.9
- net at J15.2 (Pin_2): now also R95.1
- net at U4.1 (ADJ): now also R33.2
- net at U4.2 (VO): now also R33.1
- net at U6.13 (CP): now also R36.1
- net at U16.2: now also Q2.2 (S)
- net at D15.2 (A): now also U15.4 (IP1)
- net at C19.1: now also U14.1 (Bootstrap)
- net at U15.9 (DTACKN): now also R93.1
- net at C25.1: now also U14.8 (Soft_Start)
- new net: D8.1 (K), D9.2 (A)
- new net: C22.1, Q1.2 (S)
- new net: Q1.1 (G), R34.1
- new net: Q10.2 (B), R94.1
- new net: Q4.2 (B), R96.1
- new net: Q4.1 (C), R97.2
Other:
- moved on the sheet: C1, C11, C19, C25, C43, D1, D15, D16, D17, D4, D5, J15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

Commit message: unterseite
Parts:
- removed U5: 40374, Package_DIP:DIP-20_W7.62mm, symbol 4xxx_IEEE:40374
- added U5: 74HCT574, Package_DIP:DIP-20_W7.62mm, symbol 74xx:74HCT574
- R107: now not fitted
Connections:
- net +5V: now also C2.2, C23.1, R38.2, R59.2, R91.2, U5.20 (VCC)
- net GND: now also Q11.3 (E), U5.10 (GND)
- net at R112.1: now also J17.10 (Pin_10)
- net at R104.2: now also D14.2 (A)
- net at C11.1, C43.1, L1.2: no longer C1.1
- net at R84.2: now also R51.2
- net at R35.2: now also U8.4 (AGND)
- net at R110.1: now also J17.7 (Pin_7)
- net at R47.2: now also U5.19 (Q0)
- net at R101.1: now also J16.1 (Pin_1)
- net at R101.2: now also Q5.1 (C)
- net at J5.b7 (Pin_b7): now also U3.6
- net at U3.9: now also U16.13
- net at U10.11 (B7): now also U1.9 (D7), U5.9 (D7)
- net at U10.12 (B6): now also U1.8 (D6), U5.8 (D6)
- net at U10.13 (B5): now also U1.7 (D5), U5.7 (D5)
- net at U10.14 (B4): now also U1.6 (D4), U5.6 (D4)
- net at U10.15 (B3): now also U1.5 (D3), U5.5 (D3)
- net at U10.16 (B2): now also U1.4 (D2), U5.4 (D2)
- net at U10.17 (B1): now also U1.3 (D1), U5.3 (D1)
- net at U10.18 (B0): now also U1.2 (D0), U5.2 (D0)
- net at U10.4 (A2): now also R80.2
- net at R106.1: now also J17.5 (Pin_5)
- net at R59.1: now also Q6.1 (C)
- net at R66.2: now also J20.5 (Pin_5)
- net at R115.2: now also Q12.1 (C)
- net at R105.1: now also J17.4 (Pin_4)
- net at R103.1: now also J16.2 (Pin_2)
- net at R39.2: now also J2.3 (Pin_3)
- net at R54.1: now also J14.8 (Pin_8)
- net at R86.1: now also J13.5 (Pin_5)
- net at U21.5: now also D11.2 (A), Q12.2 (B), R61.2
- net at D12.2 (A): now also R67.2
- net at J20.2 (Pin_2): now also R114.1
- net at C32.2: now also R116.2
- net at J14.6 (Pin_6): now also R53.1
- net at R114.2: now also U21.2
- net at R63.1: now also R62.1
- net at R88.1: now also J13.8 (Pin_8)
- net at Q11.1 (C): now also R100.2
- net at Q11.2 (B): now also R98.1
- net at J17.6 (Pin_6): now also R109.1
- net at J17.8 (Pin_8): now also R111.1
- net at R4.2, R6.2: now also C15.2
- net at R79.2: now also R48.2, U5.18 (Q1)
- net at R113.1: now also J18.2 (Pin_2), U19.7 (B)
- net at R85.2: now also J13.4 (Pin_4)
- net at R99.1: now also J15.3 (Pin_3)
- net at R87.1: now also J13.6 (Pin_6)
- net at R53.2: now also U5.13 (Q6)
- net at R65.1: now also U21.8
- net at U1.1 (OE): now also U5.1 (OE)
- net at R81.2: now also U5.17 (Q2)
- net at U3.13: now also U16.1
- net at J8.2 (Pin_2): now also R43.1
- net at Q12.3 (E): now also R61.1
- net at R96.2: now also U15.27 (OP4)
- net at R60.2: now also Q6.2 (B)
- net at J10.3 (Pin_3): now also R117.1
- net at R30.1: now also R41.2
- net at R52.2: now also U5.14 (Q5)
Other:
- moved on the sheet: C1, C2, C23, D11, D12, D4, D5, J10, J13, J14, J16, J17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

Commit message: power
Connections:
- net +12V: now also J16.4 (Pin_4), J21.2 (Pin_2)
- net +5V: now also D14.1 (K)
- net at R115.1: now also J20.3 (Pin_3)
- net at Q12.1 (C), R115.2: now also D11.1 (K)
- net at J20.4 (Pin_4): now also Q12.3 (E), R61.1
- net at R118.1: now also C1.1
Other:
- moved on the sheet: D11, D14, J20, J21, Q12, R104, R114, R115, R118, R61, R65, R66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
