File: Steuereinheit.kicad_sch (KiCad schematic)
At the start: 238 parts, among them J1 Tueroeffnungen, J10 Fadenfoul, J11 Netzteil, J12 Serienplan, J13 Serienplan 2, J14 Muenzeinheit 2, J15 I2C-Bus, J16 Kodierg., J17 TTL-Ein-/Ausgaenge, J18 RS485 Aus, J19 RS485 Ein, J2 PSG In/OUT, J20 Serielle-S., J21 Tuerschalter, J3 Lautsprecher, J4 DIN41612_03x10_ABC, J5 DIN41612_03x10_ABC, J6 Service, J7 Maschine, J8 Muenzeinheit, J9 Akzeptor, Q1 BSS100, Q10 BC337, Q11 BC337, Q12 BC337, Q2 BSS100, Q3 BC327, Q4 BC337, Q5 BC337, Q6 BC337, Q7 BC337, Q8 BC337, Q9 BC327, U1 74LS573, U10 74HC245, U11 SG-531, U12 74AHCT125, U13 TL7705A, U15 68C681, U16 74LS32, U17 74HC138, U18 TC428, U19 SN75176AP, U2 TS271, U20 SN75176AP, U21 LTV-827, U3 74HC02, U4 LM317L_TO92, U5 74HCT574, U6 74LS393, U7 74LS195, U8 AD7224KN, U9 YM2149

Commit message: data
Parts:
- added C27: 1u 35V, Capacitor_THT:CP_Radial_Tantal_D4.5mm_P2.50mm, symbol Device:C_Polarized
Connections:
- net +5V: now also C10.1, C11.1, C43.1, L1.2, R108.1, R16.2, R37.2, U11.8 (Vcc)
- net GND: now also C1.2, C2.1, C32.1, D8.2 (A), J4.a10 (Pin_a10), J4.a4 (Pin_a4), J4.b10 (Pin_b10), R109.2, R110.2, R111.2, R112.2, R2.1, R62.1, R63.1, R64.1, U15.33 (X2), U8.1 (VSS), C27.2
- net at C19.2, D1.1 (K), L1.1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: now also R118.2
- net at R10.1, R8.1: now also C15.1, R6.1
- net at R69.2: now also R70.2, U14.4 (P.Fail_Input)
- net D1: now reaches J5.b2 (Pin_b2)
- net D1: now also U15.16 (D1), U9.36 (DA1)
- net D4: now reaches J5.b3 (Pin_b3)
- net D4: now also U15.23 (D4), U9.33 (DA4)
- net D6: now reaches J5.b4 (Pin_b4)
- net D6: now also U15.22 (D6), U9.31 (DA6)
- net cA0: now reaches J5.b7 (Pin_b7), U3.6
- net cA3: now reaches J5.b8 (Pin_b8)
- net cA7: now reaches J5.b9 (Pin_b9)
- net at U10.1 (A->B): now also R45.2
- net at U10.9 (A7): now also R55.2
- net at R119.2: now also D6.2 (A)
- net at R5.1: now also C3.1, U2.3 (+)
- net at R12.2: now also C5.1, R11.2, R13.2, R9.2
- net at R95.2: now also R99.2
- net at U8.3 (VREF): now also R33.1, U4.2 (VO)
- net at Q6.1 (C), R59.1: now also D13.1 (K)
- net cD9: now reaches J4.b2 (Pin_b2)
- net cD12: now reaches J4.b3 (Pin_b3)
- net cD14: now reaches J4.b4 (Pin_b4)
- net cD10: now reaches J4.c2 (Pin_c2)
- net cD13: now reaches J4.c3 (Pin_c3)
- net cD15: now reaches J4.c4 (Pin_c4)
- net at U20.1 (R): now also U12.6, U19.1 (R)
- net at U14.13 (Vref): now also C18.1
- net at U14.14 (Vstart): now also C17.1
- net at U14.17 (R_Osc): now also R44.2
- net at U14.18 (C_Osc): now also C20.2
- net at U11.1 (OE): now also R37.1
- net at U2.6: now also C15.2, R4.2, R6.2
- net at U2.7 (V+): now also C4.2
- net at C32.2, R116.2: now also R62.2
- net D0: now reaches J5.a2 (Pin_a2)
- net D0: now also U15.25 (D0), U9.37 (DA0)
- net D3: now reaches J5.a3 (Pin_a3)
- net D3: now also U15.17 (D3), U9.34 (DA3)
- net cRW: now reaches J5.a5 (Pin_a5)
- net cCLKOUT: now reaches J5.a6 (Pin_a6), R14.2
- net cA2: now reaches J5.a8 (Pin_a8)
- net cA6: now reaches J5.a9 (Pin_a9)
- net at R100.1: now also J15.3 (Pin_3), R99.1
- net at J3.4 (Pin_4): now also R4.1
- net at J3.6 (Pin_6), R15.2: now also R21.2
- net D2: now reaches J5.c2 (Pin_c2)
- net D2: now also U15.24 (D2), U9.35 (DA2)
- net D5: now reaches J5.c3 (Pin_c3)
- net D5: now also U15.18 (D5), U9.32 (DA5)
- net D7: now reaches J5.c4 (Pin_c4)
- net D7: now also U15.19 (D7), U9.30 (DA7)
- net cRESET: now reaches J5.c5 (Pin_c5)
- net cA1: now reaches J5.c7 (Pin_c7)
- net cA5: now reaches J5.c8 (Pin_c8)
- net cA8: now reaches J5.c9 (Pin_c9)
- net cD8: now reaches J4.a2 (Pin_a2)
- net cD11: now reaches J4.a3 (Pin_a3)
- net at R14.1: now also U7.1 (~{MR}), U7.9 (~{PE})
- net at U6.11 (Q0): now also U9.22 (CLOCK)
- net at U16.4: now also U16.5
- net at U3.11: now also U3.12
- net A4: now reaches U15.1 (A1)
- net A1: now reaches U15.3 (A2)
- net A2: now reaches U15.5 (A3)
- net A3: now reaches U15.6 (A4)
- net at U9.29 (BC1): now also U3.4
- no-connect marks 0 -> 1
Other:
- moved on the sheet: C1, C10, C15, C17, C18, C19, C20, C25, C3, C30, C32, C34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
