File: Steuereinheit.kicad_sch (KiCad schematic)
At the start: 239 parts, among them J1 Tueroeffnungen, J10 Fadenfoul, J11 Netzteil, J12 Serienplan, J13 Serienplan 2, J14 Muenzeinheit 2, J15 I2C-Bus, J16 Kodierg., J17 TTL-Ein-/Ausgaenge, J18 RS485 Aus, J19 RS485 Ein, J2 PSG In/OUT, J20 Serielle-S., J21 Tuerschalter, J3 Lautsprecher, J4 DIN41612_03x10_ABC, J5 DIN41612_03x10_ABC, J6 Service, J7 Maschine, J8 Muenzeinheit, J9 Akzeptor, Q1 BSS100, Q10 BC337, Q11 BC337, Q12 BC337, Q2 BSS100, Q3 BC327, Q4 BC337, Q5 BC337, Q6 BC337, Q7 BC337, Q8 BC337, Q9 BC327, U1 74LS573, U10 74HC245, U11 SG-531, U12 74AHCT125, U13 TL7705A, U15 68C681, U16 74LS32, U17 74HC138, U18 TC428, U19 SN75176AP, U2 TS271, U20 SN75176AP, U21 LTV-827, U3 74HC02, U4 LM317L_TO92, U5 74HCT574, U6 74LS393, U7 74LS195, U8 AD7224KN, U9 YM2149

Commit message: vorne
Connections:
- net cRESET is gone; now on net RESET: J5.c5 (Pin_c5)
- net +5V: now also R113.2, R56.1, R92.2, R93.2, R95.2, R99.2, U4.3 (VI)
- net GND: now also R25.2, R26.2, R28.2
- net at R18.1, U6.12 (MR), U6.2 (MR): now also U17.4 (~{E0})
- net IOA0: now reaches J17.10 (Pin_10), R112.1
- net IOA0: now also U9.21 (IOA0)
- net cMISO: now reaches R104.1
- net cMISO: now also J16.2 (Pin_2), R103.1
- net MISO: now reaches D14.2 (A), R104.2
- net at R35.2, U8.4 (AGND): now also R33.2, R34.2, U4.1 (ADJ)
- net at D4.1 (K): now also U3.8
- net at D4.2 (A), D5.2 (A): now also J5.b5 (Pin_b5)
- net MOSI: now reaches J16.1 (Pin_1), R101.1
- net at U10.3 (A1): now also J13.4 (Pin_4), R85.2
- net at D6.2 (A), R119.2: now also U7.6 (P2)
- net at C26.1: now also U13.1 (REF)
- net at R54.2: now also R46.2, R82.2
- net at J19.1 (Pin_1), U20.6 (A): now also R58.1
- net at R63.2: now also R117.2
- net at J3.2 (Pin_2): now also R1.1
- net at R102.2: now also U15.13 (OP3)
- net IOA7: now reaches U9.14 (IOA7)
- net IOA6: now reaches U9.15 (IOA6)
- net IOA5: now reaches U9.16 (IOA5)
- net IOA4: now reaches U9.17 (IOA4)
- net IOA3: now reaches U9.18 (IOA3)
- net IOA2: now reaches U9.19 (IOA2)
- net IOA1: now reaches U9.20 (IOA1)
- net RESET: now reaches U9.23 (~{RESET})
Other:
- moved on the sheet: C22, C26, D14, D4, D5, D6, J13, Q1, Q2, Q5, R1, R101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

Commit message: widerstände reihenfolge
Parts:
- renumbered R15 to R14, R14 to R15
Connections:
- net +5V: now also R15.1; no longer R21.1
- net cCLKOUT: now also R21.2; no longer R15.2
- net at Q7.1 (C): now also R71.1
- net at J9.3 (Pin_3): now also R76.1
- net at U10.5 (A3): now also R89.1
- net at U10.6 (A4): now also R90.1
- net at J3.6 (Pin_6), R14.2: now also R15.2; no longer R21.2
- net at U7.1 (~{MR}), U7.9 (~{PE}): now also R21.1; no longer R15.1
- net at R76.2: now also D15.2 (A), U15.4 (IP1)
Other:
- moved on the sheet: C18, C20, D15, Q7, R15, R21, R44, R76, R89, R90

Commit message: IO
Connections:
- net GND: now also Q8.3 (E)
- net RESET: now also U8.17 (~{RST})
- net at Q7.2 (B): now also Q8.1 (C)
- net at Q3.2 (B): now also U15.14 (OP5)
- net at U3.2: now also U15.8 (RWN)
- net at Q10.1 (C): now also R93.1, U15.9 (DTACKN)
- net at Q8.2 (B): now also R73.1
- net at Q9.2 (B): now also U15.26 (OP6)
- net IOB3: now reaches U9.10 (IOB3)
- net IOB2: now reaches U9.11 (IOB2)
- net IOB1: now reaches U9.12 (IOB1)
- net IOB0: now reaches U9.13 (IOB0)
- net IOB7: now reaches U9.6 (IOB7)
- net IOB6: now reaches U9.7 (IOB6)
- net IOB5: now reaches U9.8 (IOB5)
- net IOB4: now reaches U9.9 (IOB4)
Other:
- moved on the sheet: D16, D17, Q10, Q3, Q8, Q9, R73, R92, R94, U16E

Commit message: serienplan
Connections:
- net D0: now also U8.13 (DB0(LSB))
- net D1: now also U8.12 (DB1)
- net D2: now also U8.11 (DB2)
- net D3: now also U8.10 (DB3)
- net D4: now also U8.9 (DB4)
- net D5: now also U8.8 (DB5)
- net D6: now also U8.7 (DB6)
- net D7: now also U8.6 (DB7(MSB))
- net cA7: now also U17.2 (A1)
- net cA8: now also U17.3 (A2)
- net cD8: now also J17.7 (Pin_7), R110.1
- net at R84.1: now also J13.3 (Pin_3)
- net at R83.1: now also J13.2 (Pin_2)
- net at D8.1 (K), D9.2 (A): now also J5.c6 (Pin_c6), U13.3 (CT), U13.5 (~{RESET})
- net at R80.2, U10.4 (A2): now also J12.4 (Pin_4)
- net at J4.c8 (Pin_c8): now also U15.37 (IACKN)
- net at R88.2: now also U18.5 (OUT_B)
- net at U18.2 (IN_A): now also U15.15 (OP7)
- net at R79.1: now also J12.5 (Pin_5)
- net at R82.1: now also J12.8 (Pin_8)
- net at R81.1: now also J12.6 (Pin_6)
- net at J12.2 (Pin_2): now also R77.1
- net at J12.3 (Pin_3): now also R78.1
Other:
- moved on the sheet: D8, D9, J12, R51, R77, R78, R83, R84, U18

Commit message: vorderseite und verdrahtungsplan
Connections:
- net cA2 is gone; now on net A2: J5.a8 (Pin_a8)
- net cA3 is gone; now on net A3: J5.b8 (Pin_b8)
- net +12V: now also J10.2 (Pin_2), J2.6 (Pin_6)
- net +24V: now also C42.2
- net +5V: now also D15.1 (K), U14.9 (Feedback_In.), U21.3
- net D0: now also U1.2 (D0), U10.18 (B0), U5.2 (D0)
- net D1: now also U1.3 (D1), U10.17 (B1), U5.3 (D1)
- net D2: now also U1.4 (D2), U10.16 (B2), U5.4 (D2)
- net D3: now also U1.5 (D3), U10.15 (B3), U5.5 (D3)
- net D4: now also U1.6 (D4), U10.14 (B4), U5.6 (D4)
- net D5: now also U1.7 (D5), U10.13 (B5), U5.7 (D5)
- net D6: now also U1.8 (D6), U10.12 (B6), U5.8 (D6)
- net D7: now also U1.9 (D7), U10.11 (B7), U5.9 (D7)
- net GND: now also Q6.3 (E), R60.1, U20.3 (DE); no longer C3.2, C4.1, R7.2, U2.4 (V-)
- net IOA1: now also J17.8 (Pin_8), R111.1
- net IOA2: now also J17.7 (Pin_7), R110.1
- net IOA3: now also J17.6 (Pin_6), R109.1
- net IOA7: now also J1.4 (Pin_4), R24.1
- net IOB6: now also R23.1
- net IOB7: now also R22.1
- net RESET: now also D8.1 (K), D9.2 (A), J10.3 (Pin_3), J5.c6 (Pin_c6), R117.1, U13.3 (CT), U13.5 (~{RESET}), U14.3 (Reset_Out), U15.34 (RESETN)
- net cA6: now also U17.1 (A0)
- net cD8: no longer J17.7 (Pin_7), R110.1
- net at U6.5 (Q2): now also U15.36 (IP2), U15.38 (IP5)
- net EXTRES: now reaches R74.1
- net EXTRES: now also J11.2 (Pin_2)
- net at R2.2: now also U1.1 (OE), U5.1 (OE)
- net ENSFI: now reaches J9.2 (Pin_2), R71.2
- net MISFI: now reaches J9.3 (Pin_3), R76.1
- net ANZ2: now reaches J13.3 (Pin_3), R84.1
- net at R51.2, R84.2: now also U1.15 (Q4)
- net MUX2: now reaches J13.2 (Pin_2), R83.1
- net at R83.2: now also U1.16 (Q3)
- net EnMa: now reaches R47.1
- net EnMa: now also J7.6 (Pin_6)
- net 2MA: now reaches R50.1
- net 2MA: now also J7.2 (Pin_2)
- net at R50.2: now also U1.13 (Q6)
- net at R20.1, U12.1: now also U12.4
- net at R91.1: now also D16.2 (A)
- net at U16.13, U3.9: now also J4.c9 (Pin_c9)
- net at U10.19 (CE): now also U16.8
- net OUTT2: now reaches J13.4 (Pin_4), R85.2, U10.3 (A1)
- net OUTT: now reaches J12.4 (Pin_4), R80.2, U10.4 (A2)
- net LI2: now reaches R89.1, U10.5 (A3)
- net LI2: now also J14.4 (Pin_4)
- net EMP2: now reaches R90.1, U10.6 (A4)
- net EMP2: now also J14.5 (Pin_5)
- net OUTB0: now reaches J17.5 (Pin_5), R106.1
- net at R12.1: now also U9.4 (B)
- net SCL: now reaches J15.2 (Pin_2), R95.1
- net at U8.14 (~{CS}): now also D6.1 (K), U8.16 (~{LDAC})
- net SpZa: now reaches J20.5 (Pin_5), R66.2
- net TUERK: now reaches J4.b6 (Pin_b6)
- net TUERK: now also C4.2, D3.1 (K), J1.2 (Pin_2), J21.1 (Pin_1), U2.7 (V+)
- net TXDT: now reaches J20.3 (Pin_3), R115.1
- net OUTB1: now reaches J17.4 (Pin_4), R105.1
- net ME2: now reaches R51.1
- net ME2: now also J14.2 (Pin_2)
- net SpZaTTL: now reaches J2.3 (Pin_3), R39.2
- net DataST: now reaches J6.2 (Pin_2)
- net DataST: now also R32.2
- net nTaktST: now reaches J6.3 (Pin_3), R30.2
- net EnST: now reaches J6.4 (Pin_4), R31.2
- net OUTST: now reaches J6.5 (Pin_5), R28.1
- net nTME2: now reaches J14.8 (Pin_8), R54.1
- net at J4.c6 (Pin_c6): now also U17.14 (~{Y1})
- net at U14.2 (Reset_Delay): now also C24.1
- net at U14.7 (Freq._Comp.): now also C28.1, C29.2
- net EMUX2: now reaches J13.5 (Pin_5), R86.1
- net at R19.1, U7.15 (Q0): now also U17.6 (E2), U7.7 (P3)
- net CLOCK: now reaches U11.5 (OUT)
- net CLOCK: now also R36.1, U15.32 (X1/CLK), U6.13 (CP)
- net SCK: now reaches J1.5 (Pin_5), R23.2
- net at U17.11 (~{Y4}): now also U16.9
- net at U17.12 (~{Y3}): now also D5.1 (K), U16.12
- net at U17.9 (~{Y6}): now also U15.35 (CSN)
- net RXDT: now reaches J20.2 (Pin_2), R114.1
- net at U12.13: now also R108.2
- net AW2: now reaches J14.3 (Pin_3)
- net AW2: now also R52.1
- net EnME2: now reaches J14.6 (Pin_6), R53.1
- net at U5.11 (Cp): now also U16.11
- net at U5.15 (Q4): now also R87.2
- net at R81.2, U5.17 (Q2): now also R31.1
- net PSGInA5: now reaches J2.1 (Pin_1), R25.1
- net PSGInA4: now reaches J2.2 (Pin_2), R26.1
- net PSGInA4: now also U12.5
- net Data3OUT: now reaches J2.4 (Pin_4), R27.1
- net nTSP2: now reaches J13.8 (Pin_8), R88.1
- net OUTB3: now reaches J17.2 (Pin_2)
- net OUTB2: now reaches J17.3 (Pin_3)
- net SDA: now reaches J15.3 (Pin_3), R100.1, R99.1
- net +12VA: now reaches J3.1 (Pin_1)
- net +12VA: now also D3.2 (A)
- net LS_ALARM: now reaches J3.2 (Pin_2), R1.1
- net LS_KNACK: now reaches J3.3 (Pin_3)
- net LS_SOUND: now reaches J3.4 (Pin_4), R4.1
- net GNDA: now reaches J3.5 (Pin_5)
- net GNDA: now also C3.2, C4.1, R7.2, U2.4 (V-)
- net LS_5V: now reaches J3.6 (Pin_6), R14.2, R15.2
- net at R32.1: now also R49.2, U1.19 (Q0)
- net EMUX: now reaches J12.5 (Pin_5), R79.1
- net at R27.2: now also U1.14 (Q5)
- net at J4.a6 (Pin_a6): now also U15.7 (IP0)
- net at J4.a8 (Pin_a8): now also U15.21 (INTRN)
- net at J4.a9 (Pin_a9): now also U16.10
- net nTSP: now reaches J12.8 (Pin_8), R82.1
- net at J18.1 (Pin_1), U19.6 (A): now also R57.2
- net AW: now reaches R40.1
- net AW: now also J8.3 (Pin_3)
- net EANZ2: now reaches J13.6 (Pin_6), R87.1
- net at R38.1: now also U13.2 (~{RESIN})
- net at U3.3: now also U3.5
- net 1MA: now reaches J7.3 (Pin_3)
- net 1MA: now also R49.1
- net OUTMA: now reaches J7.4 (Pin_4)
- net MUXMA: now reaches J7.5 (Pin_5)
- net MUXMA: now also R48.1
- net nTMA: now reaches J7.8 (Pin_8)
- net nTMA: now also R46.1
- net at U1.12 (Q7): now also R43.2
- net EANZ: now reaches J12.6 (Pin_6), R81.1
- net at U16.4, U16.5: now also U15.30 (TXDA)
- net at R13.1: now also U9.3 (A)
- net at R98.2: now also Q9.2 (B), U15.26 (OP6)
- net ME: now reaches J8.2 (Pin_2), R43.1
- net OUTLI: now reaches J8.4 (Pin_4)
- net OUTLI: now also R64.2
- net OUTEMP: now reaches J8.5 (Pin_5), R29.1
- net EnME: now reaches J8.6 (Pin_6)
- net EnME: now also R42.1
- net nTME: now reaches J8.8 (Pin_8)
- net nTME: now also R41.1
- net at C29.1: now also R68.2
- net TUER: now reaches J21.3 (Pin_3)
- net TUER: now also R116.1
- net at R72.2: now also D15.2 (A), R76.2, U15.4 (IP1)
- net at U21.7: now also Q6.2 (B), R60.2
- net SOUT: now reaches J1.3 (Pin_3), R22.2
- net MUX: now reaches J12.2 (Pin_2), R77.1
- net ANZ: now reaches J12.3 (Pin_3), R78.1
- net at R11.1: now also U9.38 (C)
- net FREI: now reaches J10.1 (Pin_1)
- net at R17.1: now also U15.28 (OP2)
- net MOSI renamed OD
- net cMISO renamed SID
Other:
- moved on the sheet: C13, C15, C16, C2, C21, C23, C24, C28, C29, C3, C32, C33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

Commit message: fertig?
Parts:
- added JP1, JP2: Jumper_2_Bridged, Jumper:SolderJumper-2_P1.3mm_Bridged_Pad1.0x1.5mm, symbol Jumper:Jumper_2_Bridged
- C11, C34, C43: footprint Capacitor_THT:CP_Radial_D8.0mm_P5.00mm -> Capacitor_THT:CP_Radial_D12.5mm_P5.00mm
- J1: value Tueroeffnungen -> Tueroeffn.
- J13: value Serienplan 2 -> Serienplan II
- J14: value Muenzeinheit 2 -> Muenzeinheit II
- J15: value I2C-Bus -> I2C Bus
- J17: value TTL-Ein-/Ausgaenge -> PSG-Port
- J18: value RS485 Aus -> In
- J19: value RS485 Ein -> Out
- J2: value PSG In/OUT -> PSGIn/Out
- J20: value Serielle-S. -> Seriell-TTL/Spz
- J21: value Tuerschalter -> Tuersch.
- J6: value Service -> Service-Tast.
- U4: value LM317L_TO92 -> LM317LZ
Connections:
- net A1 is gone; now on net cA1: U15.3 (A2)
- net A4 is gone; now on net cA0: U15.1 (A1)
- net IOA4 is gone; now on net OUTB2: U9.17 (IOA4)
- net IOA5 is gone; now on net OUTB3: U9.16 (IOA5)
- net PSGInA5 is gone; now on net OUTB3: J2.1 (Pin_1), R25.1
- net +12VA: now also C16.1, C4.2, D3.1 (K), U2.7 (V+), U4.3 (VI), U8.18 (VDD); no longer D3.2 (A), J3.1 (Pin_1)
- net +5V: no longer C16.1, U4.3 (VI), U8.18 (VDD)
- net D1: now also U1.8 (D6), U10.12 (B6), U5.8 (D6); no longer U1.3 (D1), U10.17 (B1), U5.3 (D1)
- net D2: now also U1.9 (D7), U10.11 (B7), U5.9 (D7); no longer U1.4 (D2), U10.16 (B2), U5.4 (D2)
- net D3: now also U1.7 (D5), U10.13 (B5), U5.7 (D5); no longer U1.5 (D3), U10.15 (B3), U5.5 (D3)
- net D4: now also U1.4 (D2), U10.16 (B2), U5.4 (D2); no longer U1.6 (D4), U10.14 (B4), U5.6 (D4)
- net D5: now also U1.3 (D1), U10.17 (B1), U5.3 (D1); no longer U1.7 (D5), U10.13 (B5), U5.7 (D5)
- net D6: now also U1.6 (D4), U10.14 (B4), U5.6 (D4); no longer U1.8 (D6), U10.12 (B6), U5.8 (D6)
- net D7: now also U1.5 (D3), U10.15 (B3), U5.5 (D3); no longer U1.9 (D7), U10.11 (B7), U5.9 (D7)
- net GND: now also Q5.3 (E), R24.2, JP1.1 (A), JP2.1 (A); no longer R9.1
- net GNDA: now also R9.1, JP1.2 (B), JP2.2 (B)
- net IOA6: now also R117.2, R63.2
- net IOB0: now also R106.2
- net IOB1: now also R105.2
- net IOB2: now also R107.2
- net IOB3: now also Q2.2 (S), R108.2, U12.13, U16.2
- net IOB4: now also U19.3 (DE)
- net IOB5: now also R65.2, U20.2 (~{RE}), U3.11, U3.12
- net LS_KNACK: now also R17.2
- net MISO: now also U15.2 (IP3)
- net OUTB2: now also J2.2 (Pin_2), R26.1
- net OUTEMP: now also U10.8 (A6), U12.5
- net OUTLI: now also U10.2 (A0)
- net OUTMA: now also R55.2, U10.9 (A7)
- net OUTST: now also U10.7 (A5)
- net RESET: now also C27.1, R74.2; no longer J10.3 (Pin_3), J5.c5 (Pin_c5), R117.1, U15.34 (RESETN), U8.17 (~{RST}), U9.23 (~{RESET})
- net SCL: now also R97.1
- net TUERK: no longer C4.2, D3.1 (K), U2.7 (V+)
- net cD8: now also U12.8
- net cRW: now also U15.8 (RWN), U3.2
- net at U6.1 (CP): now also R21.1, U7.1 (~{MR}), U7.9 (~{PE})
- net at R18.1, U17.4 (~{E0}), U6.12 (MR)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: now also U9.24 (~{A9})
- net at Q7.2 (B), Q8.1 (C): now also R75.1
- net at R47.2, U5.19 (Q0): now also R42.2
- net at R20.1, U12.1, U12.4: now also Q2.1 (G)
- net at D4.1 (K), U3.8: now also U16.9, U17.11 (~{Y4})
- net at D4.2 (A), D5.2 (A), J5.b5 (Pin_b5): now also Q10.1 (C), R93.1, U15.9 (DTACKN)
- net DB_RESET: now reaches D9.1 (K)
- net DB_RESET: now also J10.3 (Pin_3), R117.1
- net at J5.b6 (Pin_b6): now also U17.13 (~{Y2})
- net at U3.10: now also U1.11 (Load), U7.14 (Q1)
- net at J4.c9 (Pin_c9), U16.13, U3.9: now also U8.15 (~{WR})
- net at U10.19 (CE), U16.8: now also U12.10
- net at R119.1: now also U17.10 (~{Y5}), U3.3, U3.5
- net at D6.1 (K), U8.14 (~{CS}), U8.16 (~{LDAC}): now also U17.15 (~{Y0})
- net at U8.2 (VOUT): now also C6.1
- net at D13.1 (K), Q6.1 (C), R59.1: now also U15.31 (RXDA)
- net at R66.1: now also R39.1, U18.7 (~{OUT_A})
- net at J4.b9 (Pin_b9): now also U17.5 (~{E1})
- net at R46.2, R54.2, R82.2: now also R30.1, R41.2, R88.2, U18.5 (OUT_B)
- net at U12.6, U19.1 (R), U20.1 (R): now also U15.10 (RXDB)
- net at R86.2: now also U5.16 (Q3)
- net at U21.4: now also D12.1 (K), R67.1
- net at U21.6: now also J20.1 (Pin_1), U21.1
- net at U2.8 (Subst.): now also R7.1
- net at D12.2 (A), R67.2: now also U16.6
- net at C22.1, Q1.2 (S): now also R107.1
- net at C32.2, R116.2, R62.2: now also U15.39 (IP4)
- net at U12.11, U12.3: now also R40.2
- net at U12.12: now also U5.12 (Q7)
- net at Q11.1 (C), R100.2: now also J4.a6 (Pin_a6), U15.7 (IP0)
- net at U18.4 (IN_B): now also U7.2 (J)
- net at U12.2: now also U15.11 (TXDB), U19.4 (D)
- net at Q5.2 (B): now also R102.1
- net INTRN: now reaches J4.a8 (Pin_a8), U15.21 (INTRN)
- net INTRN: now also R16.1
- net at U19.2 (~{RE}): now also U16.3
- net at U1.17 (Q2): now also R78.2
- net at U1.18 (Q1): now also R77.2
- net at U7.3 (~{K}): now also R94.2
- net at Q6.2 (B), R60.2, U21.7: now also D13.2 (A)
- net at R1.2: now also U15.29 (OP0)
- net at U15.12 (OP1): now also R73.2
- net A2 renamed cA2
- net A3 renamed cA3
- removed net PSGInA4: J2.2 (Pin_2), R26.1, U12.5
- new net: D3.2 (A), J3.1 (Pin_1)
- new net nRESET: J5.c5 (Pin_c5), U15.34 (RESETN), U8.17 (~{RST}), U9.23 (~{RESET})
- no-connect marks 1 -> 27
Other:
- note added: "PINS 2&3 ARE SWAPPED ON L317LZ"
- moved on the sheet: C32, D12, D3, J21, J7, Q10, Q2, Q7, Q8, R107, R116, R16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

Commit message: op pins
Parts:
- D16: value LED -> SDA_LED
Connections:
- net OP5: now reaches Q3.2 (B), U15.14 (OP5)
- net OP7: now reaches U15.15 (OP7), U18.2 (IN_A)
- net OP3: now reaches R102.2, U15.13 (OP3)
- net OP6: now reaches Q9.2 (B), R98.2, U15.26 (OP6)
- net OP4: now reaches R96.2, U15.27 (OP4)
- net OP0: now reaches R1.2, U15.29 (OP0)
- net OP2: now reaches R17.1, U15.28 (OP2)
- net OP1: now reaches R73.2, U15.12 (OP1)
Other:
- note added: "Eingaenge"
- note added: "Serienplan / Muenzeinheit I"
- note added: "Serienplan / Muenzeinheit II"
- moved on the sheet: C12, C14, C15, C23, C26, C27, C3, C30, C31, C33, C34, C35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

Commit message: notes
Connections:
- net at C15.1, R10.1, R6.1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: now also U2.2 (-)
- net Y4: now reaches D4.1 (K), U16.9, U17.11 (~{Y4}), U3.8
- net DTACKN: now reaches D4.2 (A), D5.2 (A), J5.b5 (Pin_b5), Q10.1 (C), R93.1, U15.9 (DTACKN)
- net Y2: now reaches J5.b6 (Pin_b6), U17.13 (~{Y2})
- net EN_YM: now reaches R119.1, U17.10 (~{Y5}), U3.3, U3.5
- net EN_DAC: now reaches D6.1 (K), U17.15 (~{Y0}), U8.14 (~{CS}), U8.16 (~{LDAC})
- net DB_RX: now reaches J4.b8 (Pin_b8)
- net E1: now reaches J4.b9 (Pin_b9), U17.5 (~{E1})
- net Y1: now reaches J4.c6 (Pin_c6), U17.14 (~{Y1})
- net DB_TX: now reaches J4.c7 (Pin_c7)
- net IACKN: now reaches J4.c8 (Pin_c8), U15.37 (IACKN)
- net Y3: now reaches D5.1 (K), U16.12, U17.12 (~{Y3})
- net EN_UART: now reaches U15.35 (CSN), U17.9 (~{Y6})
- net IP0: now reaches J4.a6 (Pin_a6), Q11.1 (C), R100.2, U15.7 (IP0)
- no-connect marks 27 -> 24
Other:
- note added: "FROM A TO B"
- moved on the sheet: U3C
