File: Steuereinheit.kicad_sch (KiCad schematic)
At the start: 242 parts, among them J1 Tueroeffn., J10 Fadenfoul, J11 Netzteil, J12 Serienplan, J13 Serienplan II, J14 Muenzeinheit II, J15 I2C Bus, J16 Kodierg., J17 PSG-Port, J18 In, J19 Out, J2 PSGIn/Out, J20 Seriell-TTL/Spz, J21 Tuersch., J3 Lautsprecher, J4 DIN41612_03x10_ABC, J5 DIN41612_03x10_ABC, J6 Service-Tast., J7 Maschine, J8 Muenzeinheit, J9 Akzeptor, Q1 BSS100, Q10 BC337, Q11 BC337, Q12 BC337, Q2 BSS100, Q3 BC327, Q4 BC337, Q5 BC337, Q6 BC337, Q7 BC337, Q8 BC337, Q9 BC327, U1 74HC573, U10 74HC245, U11 SG-531, U12 74HC125, U13 TL7705A, U15 68C681, U16 74LS32, U17 74HC138, U18 TC428, U19 SN75176AP, U2 TS271, U20 SN75176AP, U21 LTV-827, U3 74HC02, U4 LM317LZ, U5 74HC574, U6 74HC393, U7 74HC4015, U8 AD7224KN, U9 YM2149

Commit message: label
Parts:
- R55: value 47 -> 470
- TP1: value EN_YM -> EnYM; footprint TestPoint:TestPoint_THTPad_D1.0mm_Drill0.5mm -> TestPoint:TestPoint_Pad_D1.0mm
Connections:
- net EnIN: now reaches U10.19 (CE), U12.10, U16.8
- net RXDB: now reaches U12.6, U15.10 (RXDB), U19.1 (R), U20.1 (R)
- net OP6_SDA: now reaches Q11.2 (B), R98.1
- net nTakt: now reaches U18.4 (IN_B), U7.2 (Q4)
- net TXDB: now reaches U12.2, U15.11 (TXDB), U19.4 (D)
- net OP3_OD: now reaches Q5.2 (B), R102.1
- net OP4_SCL: now reaches Q4.2 (B), R96.1
- net OP1_ENSFI: now reaches Q8.2 (B), R73.1
- net CSN renamed EnUART
- net EANZ renamed EnANZ
- net EANZ2 renamed EnANZ2
- net EMUX renamed EnMUX
- net EMUX2 renamed EnMUX2
- net EN_DAC renamed EnDAC
- net EN_YM renamed EnYM
- net IOA7 renamed SIN
- net OP5 renamed OP5_LED
- net OP7 renamed nSpZ
- net OUTB0 renamed OutB0
- net OUTB1 renamed OutB1
- net OUTB2 renamed OutB2
- net OUTB3 renamed OutB3
- net OUTEMP renamed OutEMP
- net OUTLI renamed OutLI
- net OUTMA renamed OutMA
- net OUTST renamed OutST
- net OUTT renamed OutT
- net OUTT2 renamed OutT2
- net nTMA renamed nTaktMA
- net nTME renamed nTaktME
- net nTME2 renamed nTaktME2
- net nTSP renamed nTaktSP
- net nTSP2 renamed nTaktSP2
Other:
- note added: "6x47R"
- note added: "8x470R"
- moved on the sheet: D11, D12, D13, D16, D17, D2, D3, J12, J3, J7, Q12, Q3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

Commit message: bootmode
Connections:
- net CLKOUT: now reaches R21.1, U6.1 (CP), U7.1 (CP), U7.9 (CP)
- net BOOTMODE: now reaches J4.b5 (Pin_b5)
- no-connect marks 24 -> 23
Other:
- note added: "DTACKN <--> A22 for boot mode high?"
- moved on the sheet: J8
Changed lines of the file:
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@@
 	(generator_version "9.0")
 	(paper "A1")
+	(text "DTACKN <--> A22 for boot mode high?"
+		(exclude_from_sim no)
+		(at 261.112 119.634 0)
+		(effects
+			(font
+				(size 1.27 1.27)
+			)
+		)
+	)
 	(text "Serienplan /\nMuenzeinheit II"
 		(exclude_from_sim no)
@@
 	)
 	(no_connect
-		(at 45.72 187.96)
-	)
-	(no_connect
 		(at 45.72 193.04)
 	)
@@
 	)
 	(label "OutEMP"
-		(at 563.88 421.64 90)
+		(at 571.5 426.72 0)
 		(effects
 			(font
@@
 	)
 	(label "ME"
-		(at 571.5 421.64 90)
+		(at 571.5 434.34 0)
 		(effects
 			(font
@@
 	)
 	(label "OutLI"
-		(at 566.42 421.64 90)
+		(at 571.5 429.26 0)
 		(effects
 			(font
@@
 	)
 	(label "nTaktME"
-		(at 556.26 421.64 90)
+		(at 571.5 419.1 0)
 		(effects
 			(font
@@
 	)
 	(label "EnME"
-		(at 561.34 421.64 90)
+		(at 571.5 424.18 0)
 		(effects
 			(font
@@
 		)
 	)
+	(label "BOOTMODE"
+		(at 45.72 187.96 180)
+		(effects
+			(font
+				(size 1.27 1.27)
+			)
+			(justify right bottom)
+		)
+	)
 	(label "cA7"
 		(at 218.44 181.61 180)
@@
 		)
 	)
+	(label "CLKOUT"
+		(at 179.07 162.56 0)
+		(effects
+			(font
+				(size 1.27 1.27)
+			)
+			(justify left bottom)
+		)
+	)
 	(label "IP4"
 		(at 129.54 269.24 180)
@@
 	)
 	(label "AW"
-		(at 568.96 421.64 90)
+		(at 571.5 431.8 0)
 		(effects
 			(font
@@
 	(symbol
 		(lib_id "power:GND")
-		(at 574.04 421.64 180)
+		(at 571.5 436.88 90)
 		(unit 1)
 		(exclude_from_sim no)
@@
 		(fields_autoplaced yes)
 		(property "Reference" "#PWR029"
-			(at 574.04 415.29 0)
+			(at 577.85 436.88 0)
 			(effects
 				(font
@@
 		)
 		(property "Value" "GND"
-			(at 574.0401 417.83 90)
+			(at 575.31 436.8801 90)
 			(effects
 				(font
@@
 		)
 		(property "Footprint" ""
-			(at 574.04 421.64 0)
+			(at 571.5 436.88 0)
 			(effects
 				(font
@@
 		)
 		(property "Datasheet" ""
-			(at 574.04 421.64 0)
+			(at 571.5 436.88 0)
 			(effects
 				(font
@@
 		)
 		(property "Description" "Power symbol creates a global label with name \"GND\" , ground"
-			(at 574.04 421.64 0)
+			(at 571.5 436.88 0)
 			(effects
 				(font
@@
 	(symbol
 		(lib_id "Connector_Generic:Conn_01x08")
-		(at 566.42 426.72 270)
+		(at 566.42 429.26 180)
 		(unit 1)
 		(exclude_from_sim no)
@@
 		(fields_autoplaced yes)
 		(property "Reference" "J8"
-			(at 566.4201 429.26 0)
+			(at 563.88 429.2601 0)
 			(effects
 				(font
@@
 		)
 		(property "Value" "Muenzeinheit"
-			(at 563.8801 429.26 0)
+			(at 563.88 426.7201 0)
 			(effects
 				(font
@@
 		)
 		(property "Footprint" "Connector_PinHeader_2.54mm:PinHeader_1x08_P2.54mm_Vertical"
-			(at 566.42 426.72 0)
+			(at 566.42 429.26 0)
 			(effects
 				(font
@@
 		)
 		(property "Datasheet" "~"
-			(at 566.42 426.72 0)
+			(at 566.42 429.26 0)
 			(effects
 				(font
@@
 		)
 		(property "Description" "Generic connector, single row, 01x08, script generated (kicad-library-utils/schlib/autogen/connector/)"
-			(at 566.42 426.72 0)
+			(at 566.42 429.26 0)
 			(effects
 				(font
@@
 	(symbol
 		(lib_id "power:+5V")
-		(at 558.8 421.64 0)
+		(at 571.5 421.64 270)
 		(unit 1)
 		(exclude_from_sim no)
@@
 		(fields_autoplaced yes)
 		(property "Reference" "#PWR093"
-			(at 558.8 425.45 0)
+			(at 567.69 421.64 0)
 			(effects
 				(font
@@
 		)
 		(property "Value" "+5V"
-			(at 558.8001 418.295 90)
+			(at 574.845 421.6401 90)
 			(effects
 				(font
@@
 		)
 		(property "Footprint" ""
-			(at 558.8 421.64 0)
+			(at 571.5 421.64 0)
 			(effects
 				(font
@@
 		)
 		(property "Datasheet" ""
-			(at 558.8 421.64 0)
+			(at 571.5 421.64 0)
 			(effects
 				(font
@@
 		)
 		(property "Description" "Power symbol creates a global label with name \"+5V\""
-			(at 558.8 421.64 0)
+			(at 571.5 421.64 0)
 			(effects
 				(font

Commit message: mixer
Parts:
- C15, C5, C6, C7: footprint Capacitor_THT:C_Axial_L3.8mm_D2.6mm_P7.50mm_Horizontal -> (none)
- R10, R4, R6, R8: footprint Resistor_THT:R_Axial_DIN0207_L6.3mm_D2.5mm_P10.16mm_Horizontal -> (none)
Connections:
- net YM_AUDIO: now reaches C5.1, R11.2, R12.2, R13.2, R9.2
- net AD_AUDIO: now reaches C6.1, U8.2 (VOUT)
- net LS_AUDIO: now reaches C15.2, R4.2, R6.2, U2.6
Other:
- moved on the sheet: C12, C13, C14, C15, C16, C2, C21, C23, C3, C31, C32, C33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

Commit message: lampen
Parts:
- C15, C5, C6, C7: footprint (none) -> Capacitor_THT:C_Axial_L3.8mm_D2.6mm_P7.50mm_Horizontal
- R10, R4, R6, R8: footprint (none) -> Resistor_THT:R_Axial_DIN0207_L6.3mm_D2.5mm_P10.16mm_Horizontal
- U14: value ~ -> L4974A
Connections:
- net LoadU1: now reaches U1.11 (Load), U3.10, U7.14 (MR)
- net cA23: now reaches J4.c9 (Pin_c9), U16.13, U3.9, U8.15 (~{WR})
- net LoadU5: now reaches U16.11, U5.11 (Cp)
- net EMP2 renamed OutEMP2
- net LI2 renamed OutLI2
- net MUXMA renamed EnMUXMa
Other:
- moved on the sheet: D14, D3, J1, J10, J16, J17, J2, J3, J4A, J4C, Q2, Q5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

Commit message: A2
Parts:
- D17: value LED -> OP5_LED
- D2: value LED -> 5V_LED
- J4, J5: footprint Connector_DIN:DIN41612_C3_3x10_Female_Vertical_THT -> (none)
Connections:
- net IOB6 is gone; now on net SCK: R23.1, U9.7 (IOB6)
- net IOB7 is gone; now on net SOUT: R22.1, U9.6 (IOB7)
- net IP1 is gone; now on net MISFI: D15.2 (A), R72.2, R76.2, U15.4 (IP1)
- net MISFI: no longer J9.3 (Pin_3), R76.1
- net SCK: no longer J1.5 (Pin_5), R23.2
- net SOUT: no longer J1.3 (Pin_3), R22.2
- net UART_CLOCK: now reaches U15.36 (IP2), U15.38 (IP5), U6.5 (Q2)
- net OUT_OE: now reaches R2.2, U1.1 (OE), U5.1 (OE)
- net U1D6: now reaches R51.2, R84.2, U1.15 (Q4)
- net U1D7: now reaches R83.2, U1.16 (Q3)
- net U5D0: now reaches R42.2, R47.2, U5.19 (Q0)
- net U1D1: now reaches R50.2, U1.13 (Q6)
- net LED_R: now reaches D17.1 (K), Q3.3 (E)
- net LED_L: now reaches D16.1 (K), Q9.3 (E)
- net nTaktDist: now reaches R30.1, R41.2, R46.2, R54.2, R82.2, R88.2, U18.5 (OUT_B)
- net U5D7: now reaches R86.2, U5.16 (Q3)
- net U5D2: now reaches U12.12, U5.12 (Q7)
- net U5D1: now reaches R53.2, U5.13 (Q6)
- net U5D3: now reaches R52.2, U5.14 (Q5)
- net U5D6: now reaches R87.2, U5.15 (Q4)
- net U5D4: now reaches R31.1, R81.2, U5.17 (Q2)
- net U5D5: now reaches R48.2, R79.2, U5.18 (Q1)
- net POWER_LED: now reaches D2.2 (A), R3.2
- net U1D0: now reaches R32.1, R49.2, U1.19 (Q0)
- net U1D3: now reaches R27.2, U1.14 (Q5)
- net U1D2: now reaches R43.2, U1.12 (Q7)
- net U1D4: now reaches R78.2, U1.17 (Q2)
- net U1D5: now reaches R77.2, U1.18 (Q1)
- net HALF_CLOCK: now reaches U6.11 (Q0), U9.22 (CLOCK)
- net E0 renamed CLOCK_PD
- net E2 renamed CLOCK_PU
- net IACKN renamed IntACKn
- net IOB4 renamed EnTX
- net IOB5 renamed EnRX
- net IP4 renamed IP4_TUER
- net Y2 renamed EnGPU
- net Y3 renamed EnOut2
- net Y4 renamed EnIO
- net cA0 renamed A1
- net cA1 renamed A2
- net cA2 renamed A3
- net cA3 renamed A4
- net cA5 renamed A5
- net cA6 renamed A6
- net cA7 renamed A7
- net cA8 renamed A8
- net cRW renamed R/~{W}
- new net: J1.3 (Pin_3), R22.2
- new net cMISFI: J9.3 (Pin_3), R76.1
- new net cSCK: J1.5 (Pin_5), R23.2
Other:
- note added: "0x8000000"
- note added: "0x8000040"
- note added: "0x8000080"
- note added: "0x80000c0"
- note added: "0x8000100"
- note added: "0x8000140"
- note added: "0x8000180"
- note added: "0x80001c0"
- note added: "CLKOUT kommt vom SuS-Modul/Datenbank"
- note added: "FROM A TO B <---"
- note removed: "DTACKN <--> A22 for boot mode high?"
- note removed: "Eingaenge"
- note removed: "FROM A TO B"
- company: (none) -> stonedDiscord
- title: (none) -> Steuereinheit
- moved on the sheet: C1, C10, C11, C12, C13, C14, C15, C16, C17, C18, C19, C2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

Commit message: dnp 12v
Parts:
- C1, C11, C17, C18, C19, C20, C24, C25, C28, C29, C30, C34, C42, D1, L1, R118, R44, R68, R69, R70, U14: now not fitted
Connections:
- net INTRN renamed INTRn
- net IOB3 renamed EnMP
Other:
- moved on the sheet: D4, D5, Q2, R108, R31, R48, R79, R81, U16D, U3C
