File: Steuereinheit.kicad_pcb (KiCad board)
At the start: 2 copper layers, 259.7 x 80 mm, 241 parts, among them J1 Tueroeffn., J10 Fadenfoul, J11 Netzteil, J12 Serienplan, J13 Serienplan II, J14 Muenzeinheit II, J15 I2C Bus, J16 Kodierg., J17 PSG-Port, J18 In, J19 Out, J2 PSGIn/Out, J20 Seriell-TTL/Spz, J21 Tuersch., J3 Lautsprecher, J4 DIN41612_03x10_ABC, J5 DIN41612_03x10_ABC, J6 Service-Tast., J7 Maschine, J8 Muenzeinheit, J9 Akzeptor, Q1 BSS100, Q10 BC337, Q11 BC337, Q12 BC337, Q2 BSS100, Q3 BC327, Q4 BC337, Q5 BC337, Q6 BC337, Q7 BC337, Q8 BC337, Q9 BC327, U1 74LS573, U10 74HC245, U11 SG-531, U12 74AHCT125, U13 TL7705A, U15 68C681, U16 74LS32, U17 74HC138, U18 TC428, U19 SN75176AP, U2 TS271, U20 SN75176AP, U21 LTV-827, U3 74HC02, U4 LM317LZ, U5 74HCT574, U6 74LS393, U7 74LS195, U8 AD7224KN, U9 YM2149

Commit message: op pins
Parts:
- D16: value LED -> SDA_LED
Connections:
- net Net-(Q3-B) renamed OP5
- net Net-(Q9-B) renamed OP6
- net Net-(U15-OP0) renamed OP0
- net Net-(U15-OP1) renamed OP1
- net Net-(U15-OP2) renamed OP2
- net Net-(U15-OP3) renamed OP3
- net Net-(U15-OP4) renamed OP4
- net Net-(U15-OP7) renamed OP7

Commit message: notes
Connections:
- net Net-(D4-A) renamed /DTACKN
- net Net-(D4-K) renamed /Y4
- net Net-(D5-K) renamed /Y3
- net Net-(D6-K) renamed /EN_DAC
- net Net-(J4A-Pin_a6) renamed /IP0
- net Net-(J4B-Pin_b9) renamed /E1
- net Net-(J4C-Pin_c6) renamed /Y1
- net Net-(J4C-Pin_c8) renamed /IACKN
- net Net-(J5B-Pin_b6) renamed /Y2
- net Net-(U15-CSN) renamed /EN_UART
- net Net-(U17-~{Y5}) renamed /EN_YM
- C15 pad 1: Net-(C15-Pad1) -> Net-(U2--)
- J4 pad b8: unconnected-(J4B-Pin_b8-Padb8) -> /DB_RX
- J4 pad c7: unconnected-(J4C-Pin_c7-Padc7) -> /DB_TX
- R10 pad 1: Net-(C15-Pad1) -> Net-(U2--)
- R6 pad 1: Net-(C15-Pad1) -> Net-(U2--)
- R8 pad 1: Net-(C15-Pad1) -> Net-(U2--)
- U2 pad 2: unconnected-(U2---Pad2) -> Net-(U2--)
Routing:
- net Net-(U2--): track 0.00 -> 42.1 mm
- net Net-(C15-Pad1): track 40.7 -> 0.00 mm

Commit message: DRC
Parts:
- added TP1: EN_YM, TestPoint:TestPoint_THTPad_D1.0mm_Drill0.5mm, B.Cu at (212.1, 91.4)
- moved C9 0.13 mm to (236.3, 71.2)
- moved U4 0.13 mm to (230.4, 74.9)
Connections:
- net Net-(D12-A) renamed TX_A
- net Net-(J20-Pin_1) renamed /SS+5V
- net Net-(J20-Pin_4) renamed /SSGND
- net Net-(U18-~{OUT_A}) renamed SpZ
Routing:
- net /EN_YM: vias 4 -> 3

Commit message: noch mehr cleanup
Connections:
- net /E1 renamed /cA22
- net /EN_UART renamed /CSN
- net Net-(D13-A) renamed RX_A
- net Net-(D15-A) renamed /IP1
- net Net-(J4A-Pin_a9) renamed /cA21
- net Net-(U15-IP4) renamed /IP4
- net Net-(U17-E2) renamed /E2
- net Net-(U17-~{E0}) renamed /E0
