File: Steuereinheit.kicad_pcb (KiCad board)
At the start: 2 copper layers, 259.7 x 80 mm, 242 parts, among them J1 Tueroeffn., J10 Fadenfoul, J11 Netzteil, J12 Serienplan, J13 Serienplan II, J14 Muenzeinheit II, J15 I2C Bus, J16 Kodierg., J17 PSG-Port, J18 In, J19 Out, J2 PSGIn/Out, J20 Seriell-TTL/Spz, J21 Tuersch., J3 Lautsprecher, J4 DIN41612_03x10_ABC, J5 DIN41612_03x10_ABC, J6 Service-Tast., J7 Maschine, J8 Muenzeinheit, J9 Akzeptor, Q1 BSS100, Q10 BC337, Q11 BC337, Q12 BC337, Q2 BSS100, Q3 BC327, Q4 BC337, Q5 BC337, Q6 BC337, Q7 BC337, Q8 BC337, Q9 BC327, U1 74LS573, U10 74HC245, U11 SG-531, U12 74AHCT125, U13 TL7705A, U15 68C681, U16 74LS32, U17 74HC138, U18 TC428, U19 SN75176AP, U2 TS271, U20 SN75176AP, U21 LTV-827, U3 74HC02, U4 LM317LZ, U5 74HCT574, U6 74LS393, U7 74LS195, U8 AD7224KN, U9 YM2149

Commit message: ntakt chip
Parts:
- U1: value 74LS573 -> 74HC573
- U12: value 74AHCT125 -> 74HC125
- U5: value 74HCT574 -> 74HC574
- U6: value 74LS393 -> 74HC393
- U7: value 74LS195 -> 74HC4015

Commit message: label
Parts:
- added kibuzzard-68729E03: G***, kibuzzard-68729E03, B.Cu at (267.3, 69.2)
- added kibuzzard-68729E03: G***, kibuzzard-68729E03, B.Cu at (231.8, 65.4)
- added kibuzzard-68729E03: G***, kibuzzard-68729E03, B.Cu at (267.3, 113.7)
- added kibuzzard-68729E03: G***, kibuzzard-68729E03, B.Cu at (262.3, 65.4)
- added kibuzzard-68729E03: G***, kibuzzard-68729E03, B.Cu at (267.3, 106.7)
- added kibuzzard-68729E6A: G***, kibuzzard-68729E6A, B.Cu at (32.4, 87.6)
- added kibuzzard-68729E6A: G***, kibuzzard-68729E6A, B.Cu at (32.4, 120.7)
- added kibuzzard-68729E7B: G***, kibuzzard-68729E7B, B.Cu at (32.4, 113.0)
- added kibuzzard-68729E8F: G***, kibuzzard-68729E8F, B.Cu at (203.2, 124.5)
- added kibuzzard-68729E8F: G***, kibuzzard-68729E8F, B.Cu at (32.4, 102.9)
- added kibuzzard-68729E8F: G***, kibuzzard-68729E8F, B.Cu at (127.0, 124.5)
- added kibuzzard-68729E8F: G***, kibuzzard-68729E8F, B.Cu at (150.5, 124.5)
- added kibuzzard-68729F15: G***, kibuzzard-68729F15, B.Cu at (182.9, 124.5)
- added kibuzzard-68729F15: G***, kibuzzard-68729F15, B.Cu at (111.8, 124.5)
- added kibuzzard-68729F15: G***, kibuzzard-68729F15, B.Cu at (170.8, 124.5)
- added kibuzzard-68729F15: G***, kibuzzard-68729F15, B.Cu at (86.4, 124.5)
- added kibuzzard-68729F15: G***, kibuzzard-68729F15, B.Cu at (158.1, 124.5)
- added kibuzzard-68729F15: G***, kibuzzard-68729F15, B.Cu at (258.4, 124.5)
- added kibuzzard-68729F15: G***, kibuzzard-68729F15, B.Cu at (61.0, 124.5)
- added kibuzzard-68729F75: G***, kibuzzard-68729F75, B.Cu at (253.4, 124.5)
- added kibuzzard-68729F75: G***, kibuzzard-68729F75, B.Cu at (173.4, 124.5)
- added kibuzzard-68729FCB: G***, kibuzzard-68729FCB, B.Cu at (33.7, 74.9)
- added kibuzzard-68729FE2: G***, kibuzzard-68729FE2, B.Cu at (32.4, 80.0)
- added kibuzzard-68729FEA: G***, kibuzzard-68729FEA, B.Cu at (33.7, 72.4)
- added kibuzzard-68729FF2: G***, kibuzzard-68729FF2, B.Cu at (33.7, 69.8)
- added kibuzzard-6872A041: G***, kibuzzard-6872A041, B.Cu at (33.7, 77.5)
- added kibuzzard-6872A04E: G***, kibuzzard-6872A04E, B.Cu at (33.0, 67.3)
- added kibuzzard-6872A065: G***, kibuzzard-6872A065, B.Cu at (32.4, 90.2)
- added kibuzzard-6872A06E: G***, kibuzzard-6872A06E, B.Cu at (32.4, 92.7)
- added kibuzzard-6872A088: G***, kibuzzard-6872A088, B.Cu at (33.7, 95.2)
- added kibuzzard-6872A091: G***, kibuzzard-6872A091, B.Cu at (34.3, 97.8)
- added kibuzzard-6872A099: G***, kibuzzard-6872A099, B.Cu at (33.0, 100.3)
- added kibuzzard-6872A0A4: G***, kibuzzard-6872A0A4, B.Cu at (33.0, 105.4)
- added kibuzzard-6872A0AF: G***, kibuzzard-6872A0AF, B.Cu at (33.0, 115.6)
- added kibuzzard-6872A0B8: G***, kibuzzard-6872A0B8, B.Cu at (33.0, 118.1)
- added kibuzzard-6872A0D0: G***, kibuzzard-6872A0D0, B.Cu at (45.7, 122.6)
- added kibuzzard-6872A111: G***, kibuzzard-6872A111, B.Cu at (63.5, 124.5)
- added kibuzzard-6872A119: G***, kibuzzard-6872A119, B.Cu at (66.0, 124.5)
- added kibuzzard-6872A123: G***, kibuzzard-6872A123, B.Cu at (68.6, 124.5)
- added kibuzzard-6872A12C: G***, kibuzzard-6872A12C, B.Cu at (71.1, 123.2)
- added kibuzzard-6872A136: G***, kibuzzard-6872A136, B.Cu at (73.7, 123.2)
- added kibuzzard-6872A144: G***, kibuzzard-6872A144, B.Cu at (76.2, 124.5)
- added kibuzzard-6872A144: G***, kibuzzard-6872A144, B.Cu at (101.6, 124.5)
- added kibuzzard-6872A155: G***, kibuzzard-6872A155, B.Cu at (88.9, 123.8)
- added kibuzzard-6872A15D: G***, kibuzzard-6872A15D, B.Cu at (91.4, 123.8)
- added kibuzzard-6872A18D: G***, kibuzzard-6872A18D, B.Cu at (94.0, 123.8)
- added kibuzzard-6872A19B: G***, kibuzzard-6872A19B, B.Cu at (96.5, 122.6)
- added kibuzzard-6872A19E: G***, kibuzzard-6872A19E, B.Cu at (99.1, 122.6)
- added kibuzzard-6872A1B2: G***, kibuzzard-6872A1B2, B.Cu at (78.7, 122.6)
- added kibuzzard-6872A1BE: G***, kibuzzard-6872A1BE, B.Cu at (104.1, 121.9)
- added kibuzzard-6872A1D7: G***, kibuzzard-6872A1D7, B.Cu at (114.3, 124.5)
- added kibuzzard-6872A1DE: G***, kibuzzard-6872A1DE, B.Cu at (116.8, 124.5)
- added kibuzzard-6872A1E6: G***, kibuzzard-6872A1E6, B.Cu at (119.4, 124.5)
- added kibuzzard-6872A1ED: G***, kibuzzard-6872A1ED, B.Cu at (121.9, 123.8)
- added kibuzzard-6872A1F5: G***, kibuzzard-6872A1F5, B.Cu at (124.5, 123.2)
- added kibuzzard-6872A209: G***, kibuzzard-6872A209, B.Cu at (129.5, 121.9)
- added kibuzzard-6872A215: G***, kibuzzard-6872A215, B.Cu at (153.0, 124.5)
- added kibuzzard-6872A21C: G***, kibuzzard-6872A21C, B.Cu at (155.6, 124.5)
- added kibuzzard-6872A24B: G***, kibuzzard-6872A24B, B.Cu at (165.7, 124.5)
- added kibuzzard-6872A252: G***, kibuzzard-6872A252, B.Cu at (168.3, 124.5)
- added kibuzzard-6872A278: G***, kibuzzard-6872A278, B.Cu at (43.2, 124.4)
- added kibuzzard-6872A280: G***, kibuzzard-6872A280, B.Cu at (53.3, 124.5)
- added kibuzzard-6872A286: G***, kibuzzard-6872A286, B.Cu at (50.8, 124.5)
- added kibuzzard-6872A2D1: G***, kibuzzard-6872A2D1, B.Cu at (48.3, 124.5)
- added kibuzzard-6872A326: G***, kibuzzard-6872A326, B.Cu at (185.4, 123.8)
- added kibuzzard-6872A337: G***, kibuzzard-6872A337, B.Cu at (188.0, 123.8)
- added kibuzzard-6872A33C: G***, kibuzzard-6872A33C, B.Cu at (190.5, 123.8)
- added kibuzzard-6872A344: G***, kibuzzard-6872A344, B.Cu at (193.0, 123.9)
- added kibuzzard-6872A368: G***, kibuzzard-6872A368, B.Cu at (195.6, 124.5)
- added kibuzzard-6872A375: G***, kibuzzard-6872A375, B.Cu at (198.1, 124.5)
- added kibuzzard-6872A37B: G***, kibuzzard-6872A37B, B.Cu at (200.7, 124.5)
- added kibuzzard-6872A380: G***, kibuzzard-6872A380, B.Cu at (205.7, 124.5)
- added kibuzzard-6872A3BA: G***, kibuzzard-6872A3BA, B.Cu at (214.0, 125.1)
- added kibuzzard-6872A3CC: G***, kibuzzard-6872A3CC, B.Cu at (224.2, 125.1)
- added kibuzzard-6872A444: G***, kibuzzard-6872A444, B.Cu at (233.0, 123.8)
- added kibuzzard-6872A450: G***, kibuzzard-6872A450, B.Cu at (235.6, 123.8)
- added kibuzzard-6872A456: G***, kibuzzard-6872A456, B.Cu at (238.1, 123.8)
- added kibuzzard-6872A45D: G***, kibuzzard-6872A45D, B.Cu at (240.7, 123.2)
- added kibuzzard-6872A466: G***, kibuzzard-6872A466, B.Cu at (243.2, 124.5)
- added kibuzzard-6872A46F: G***, kibuzzard-6872A46F, B.Cu at (250.8, 123.8)
- added kibuzzard-6872A486: G***, kibuzzard-6872A486, B.Cu at (255.9, 123.8)
- added kibuzzard-6872A49D: G***, kibuzzard-6872A49D, B.Cu at (267.3, 118.7)
- added kibuzzard-6872A4A7: G***, kibuzzard-6872A4A7, B.Cu at (267.3, 121.3)
- added kibuzzard-6872A4B2: G***, kibuzzard-6872A4B2, B.Cu at (266.1, 116.2)
- added kibuzzard-6872A4BB: G***, kibuzzard-6872A4BB, B.Cu at (267.3, 104.1)
- added kibuzzard-6872A4C0: G***, kibuzzard-6872A4C0, B.Cu at (267.3, 101.6)
- added kibuzzard-6872A4C7: G***, kibuzzard-6872A4C7, B.Cu at (267.3, 99.1)
- added kibuzzard-6872A4D0: G***, kibuzzard-6872A4D0, B.Cu at (266.1, 96.5)
- added kibuzzard-6872A4D7: G***, kibuzzard-6872A4D7, B.Cu at (267.3, 94.0)
- added kibuzzard-6872A4E7: G***, kibuzzard-6872A4E7, B.Cu at (267.3, 81.9)
- added kibuzzard-6872A4E7: G***, kibuzzard-6872A4E7, B.Cu at (267.3, 91.4)
- added kibuzzard-6872A4F2: G***, kibuzzard-6872A4F2, B.Cu at (267.3, 88.9)
- added kibuzzard-6872A4FD: G***, kibuzzard-6872A4FD, B.Cu at (266.1, 79.4)
- added kibuzzard-6872A50A: G***, kibuzzard-6872A50A, B.Cu at (267.3, 76.8)
- added kibuzzard-6872A510: G***, kibuzzard-6872A510, B.Cu at (267.3, 74.3)
- added kibuzzard-6872A519: G***, kibuzzard-6872A519, B.Cu at (266.7, 71.8)
- added kibuzzard-6872A52D: G***, kibuzzard-6872A52D, B.Cu at (264.8, 65.4)
- added kibuzzard-6872A53B: G***, kibuzzard-6872A53B, B.Cu at (252.1, 66.0)
- added kibuzzard-6872A545: G***, kibuzzard-6872A545, B.Cu at (254.6, 66.0)
- added kibuzzard-6872A554: G***, kibuzzard-6872A554, B.Cu at (257.2, 67.3)
- added kibuzzard-6872A55F: G***, kibuzzard-6872A55F, B.Cu at (259.7, 67.6)
- added kibuzzard-6872A576: G***, kibuzzard-6872A576, B.Cu at (244.5, 65.4)
- added kibuzzard-6872A580: G***, kibuzzard-6872A580, B.Cu at (241.9, 65.4)
- added kibuzzard-6872A5D0: G***, kibuzzard-6872A5D0, B.Cu at (239.4, 65.4)
- added kibuzzard-6872A5D9: G***, kibuzzard-6872A5D9, B.Cu at (236.9, 66.0)
- added kibuzzard-6872A5E5: G***, kibuzzard-6872A5E5, B.Cu at (234.3, 66.7)
- R55: value 47 -> 470
- TP1: value EN_YM -> EnYM; footprint TestPoint:TestPoint_THTPad_D1.0mm_Drill0.5mm -> TestPoint:TestPoint_Pad_D1.0mm
- moved C17 2.58 mm to (50.3, 89.5), turned to 0 degrees
- moved Q1 0.25 mm to (234.9, 91.2)
- moved U4 0.18 mm to (230.5, 74.8)
- moved D10 0.13 mm to (238.8, 100.5)
- moved C26 0.12 mm to (235.6, 100.3)
Connections:
- net /CSN renamed /EnUART
- net /EANZ renamed /EnANZ
- net /EANZ2 renamed /EnANZ2
- net /EMUX renamed /EnMUX
- net /EMUX2 renamed /EnMUX2
- net /EN_DAC renamed /EnDAC
- net /EN_YM renamed /EnYM
- net /LS_ALARM renamed LS_ALARM
- net /LS_KNACK renamed LS_KNACK
- net /OUTB0 renamed /OutB0
- net /OUTB1 renamed /OutB1
- net /OUTB2 renamed OutB2
- net /OUTB3 renamed OutB3
- net /OUTEMP renamed /OutEMP
- net /OUTLI renamed /OutLI
- net /OUTMA renamed /OutMA
- net /OUTST renamed /OutST
- net /OUTT renamed /OutT
- net /OUTT2 renamed /OutT2
- net /nTMA renamed /nTaktMA
- net /nTME renamed /nTaktME
- net /nTME2 renamed /nTaktME2
- net /nTSP renamed /nTaktSP
- net /nTSP2 renamed /nTaktSP2
- net IOA7 renamed SIN
- net Net-(Q11-B) renamed OP6_SDA
- net Net-(Q4-B) renamed OP4_SCL
- net Net-(Q5-B) renamed OP3_OD
- net Net-(Q8-B) renamed OP1_ENSFI
- net Net-(U10-CE) renamed /EnIN
- net Net-(U15-RXDB) renamed RXDB
- net Net-(U15-TXDB) renamed TXDB
- net Net-(U18-IN_B) renamed /nTakt
- net OP0 renamed /OP0
- net OP1 renamed /OP1
- net OP2 renamed /OP2
- net OP3 renamed /OP3
- net OP4 renamed /OP4
- net OP5 renamed OP5_LED
- net OP7 renamed nSpZ
Routing:
- net Net-(U14-Vstart): track 8.28 -> 10.9 mm
- net D3: track 260.1 -> 258.8 mm
- net +12VA: track 268.6 -> 269.9 mm
Other:
- board text removed: "https://github.com/stonedDiscord/Steuereinheit"

Commit message: bootmode
Other:
- board text added: "5V"
- board text added: "A0-A8"
- board text added: "ALARM"
- board text added: "D0-D7"
- board text added: "D8-D15"
- board text added: "GND"
- board text added: "PROFIT 300"
- board text added: "RX"
- board text added: "TX"
- board text added: "https://github.com/stonedDiscord/Steuereinheit"
