File: Steuereinheit.kicad_pcb (KiCad board)
At the start: 2 copper layers, 259.7 x 80 mm, 348 parts, among them J1 Tueroeffn., J10 Fadenfoul, J11 Netzteil, J12 Serienplan, J13 Serienplan II, J14 Muenzeinheit II, J15 I2C Bus, J16 Kodierg., J17 PSG-Port, J18 In, J19 Out, J2 PSGIn/Out, J20 Seriell-TTL/Spz, J21 Tuersch., J3 Lautsprecher, J4 DIN41612_03x10_ABC, J5 DIN41612_03x10_ABC, J6 Service-Tast., J7 Maschine, J8 Muenzeinheit, J9 Akzeptor, Q1 BSS100, Q10 BC337, Q11 BC337, Q12 BC337, Q2 BSS100, Q3 BC327, Q4 BC337, Q5 BC337, Q6 BC337, Q7 BC337, Q8 BC337, Q9 BC327, U1 74HC573, U10 74HC245, U11 SG-531, U12 74HC125, U13 TL7705A, U15 68C681, U16 74LS32, U17 74HC138, U18 TC428, U19 SN75176AP, U2 TS271, U20 SN75176AP, U21 LTV-827, U3 74HC02, U4 LM317LZ, U5 74HC574, U6 74HC393, U7 74HC4015, U8 AD7224KN, U9 YM2149

Commit message: mixer
Connections:
- net /LS_SOUND renamed LS_SOUND
- net Net-(C15-Pad2) renamed /LS_AUDIO
- net Net-(C5-Pad1) renamed YM_AUDIO
- net Net-(U6A-CP) renamed /CLKOUT
- net Net-(U8-VOUT) renamed AD_AUDIO
- J4 pad b5: unconnected-(J4B-Pin_b5-Padb5) -> /BOOTMODE

Commit message: A2
Parts:
- D17: value LED -> OP5_LED
- D2: value LED -> 5V_LED
- U14: value ~ -> L4974A
Connections:
- net /CLKOUT renamed CLKOUT
- net /DTACKN renamed DTACKN
- net /E0 renamed CLOCK_PD
- net /E2 renamed CLOCK_PU
- net /EMP2 renamed /OutEMP2
- net /EnDAC renamed EnDAC
- net /EnUART renamed EnUART
- net /EnYM renamed EnYM
- net /IACKN renamed IntACKn
- net /IP1 renamed MISFI
- net /IP4 renamed IP4_TUER
- net /LI2 renamed /OutLI2
- net /MISFI renamed /cMISFI
- net /MUXMA renamed /EnMUXMa
- net /SCK renamed /cSCK
- net /SOUT renamed Net-(J1-Pin_3)
- net /Y1 renamed Y1
- net /Y2 renamed EnGPU
- net /Y3 renamed EnOut2
- net /Y4 renamed EnIO
- net /cA0 renamed A1
- net /cA1 renamed A2
- net /cA2 renamed A3
- net /cA3 renamed A4
- net /cA5 renamed /A5
- net /cA6 renamed A6
- net /cA7 renamed A7
- net /cA8 renamed A8
- net /cRW renamed R/~{W}
- net /nTakt renamed nTakt
- net IOB4 renamed EnTX
- net IOB5 renamed EnRX
- net IOB6 renamed SCK
- net IOB7 renamed SOUT
- net Net-(D16-K) renamed /LED_L
- net Net-(D17-K) renamed /LED_R
- net Net-(D2-A) renamed /POWER_LED
- net Net-(J4C-Pin_c9) renamed /cA23
- net Net-(U1-Load) renamed LoadU1
- net Net-(U1-OE) renamed OUT_OE
- net Net-(U1-Q0) renamed /U1D0
- net Net-(U1-Q1) renamed /U1D5
- net Net-(U1-Q2) renamed /U1D4
- net Net-(U1-Q3) renamed /U1D7
- net Net-(U1-Q4) renamed /U1D6
- net Net-(U1-Q5) renamed /U1D3
- net Net-(U1-Q6) renamed /U1D1
- net Net-(U1-Q7) renamed /U1D2
- net Net-(U15-IP2) renamed UART_CLOCK
- net Net-(U18-OUT_B) renamed /nTaktDist
- net Net-(U5-Cp) renamed LoadU5
- net Net-(U5-Q0) renamed /U5D0
- net Net-(U5-Q1) renamed /U5D5
- net Net-(U5-Q2) renamed /U5D4
- net Net-(U5-Q3) renamed /U5D7
- net Net-(U5-Q4) renamed /U5D6
- net Net-(U5-Q5) renamed /U5D3
- net Net-(U5-Q6) renamed /U5D1
- net Net-(U5-Q7) renamed /U5D2
- net Net-(U6B-Q0) renamed HALF_CLOCK
Other:
- board text added: "A1-A8"
- board text removed: "A0-A8"

Commit message: dnp 12v
Connections:
- net IOB3 renamed EnMP
Changed lines of the file:
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@@
 	(net 21 "IOA3")
 	(net 22 "/cA23")
-	(net 23 "IOB3")
+	(net 23 "EnMP")
 	(net 24 "A6")
 	(net 25 "IOA1")
@@
 		(sheetname "/")
 		(sheetfile "Steuereinheit.kicad_sch")
-		(attr through_hole)
+		(attr through_hole dnp)
 		(fp_line
 			(start 1.04 0)
@@
 		(sheetname "/")
 		(sheetfile "Steuereinheit.kicad_sch")
-		(attr through_hole)
+		(attr through_hole dnp)
 		(fp_line
 			(start -1.287288 -1.335)
@@
 		(sheetname "/")
 		(sheetfile "Steuereinheit.kicad_sch")
-		(attr through_hole)
+		(attr through_hole dnp)
 		(fp_line
 			(start -2.57 -3.26)
@@
 		(sheetname "/")
 		(sheetfile "Steuereinheit.kicad_sch")
-		(attr through_hole)
+		(attr through_hole dnp)
 		(fp_line
 			(start 6.12 -1.12)
@@
 		(sheetname "/")
 		(sheetfile "Steuereinheit.kicad_sch")
-		(attr through_hole)
+		(attr through_hole dnp)
 		(fp_line
 			(start 6.12 -1.12)
@@
 		(sheetname "/")
 		(sheetfile "Steuereinheit.kicad_sch")
-		(attr through_hole)
+		(attr through_hole dnp)
 		(fp_line
 			(start 8.37 -1.37)
@@
 			(layers "*.Cu" "*.Mask")
 			(remove_unused_layers no)
-			(net 23 "IOB3")
+			(net 23 "EnMP")
 			(pinfunction "IOB3")
 			(pintype "bidirectional")
@@
 			(layers "*.Cu" "*.Mask")
 			(remove_unused_layers no)
-			(net 23 "IOB3")
+			(net 23 "EnMP")
 			(pintype "input")
 		)
@@
 		(sheetname "/")
 		(sheetfile "Steuereinheit.kicad_sch")
-		(attr through_hole)
+		(attr through_hole dnp)
 		(fp_line
 			(start 9.12 0)
@@
 		(sheetname "/")
 		(sheetfile "Steuereinheit.kicad_sch")
-		(attr through_hole)
+		(attr through_hole dnp)
 		(fp_line
 			(start -1.287288 -1.335)
@@
 		(sheetname "/")
 		(sheetfile "Steuereinheit.kicad_sch")
-		(attr through_hole)
+		(attr through_hole dnp)
 		(fp_line
 			(start 6.46 0)
@@
 			(layers "*.Cu" "*.Mask")
 			(remove_unused_layers no)
-			(net 23 "IOB3")
+			(net 23 "EnMP")
 			(pintype "passive")
 		)
@@
 			(layers "*.Cu" "*.Mask")
 			(remove_unused_layers no)
-			(net 23 "IOB3")
+			(net 23 "EnMP")
 			(pintype "input")
 		)
@@
 		(sheetname "/")
 		(sheetfile "Steuereinheit.kicad_sch")
-		(attr through_hole)
+		(attr through_hole dnp)
 		(fp_line
 			(start -4.317082 -3.575)
@@
 		(sheetname "/")
 		(sheetfile "Steuereinheit.kicad_sch")
-		(attr through_hole)
+		(attr through_hole dnp)
 		(fp_line
 			(start 8.37 -1.37)
@@
 		(sheetname "/")
 		(sheetfile "Steuereinheit.kicad_sch")
-		(attr through_hole)
+		(attr through_hole dnp)
 		(fp_line
 			(start 0.485 0.92)
@@
 		(sheetname "/")
 		(sheetfile "Steuereinheit.kicad_sch")
-		(attr through_hole)
+		(attr through_hole dnp)
 		(fp_line
 			(start -4.317082 -3.575)
@@
 		(sheetname "/")
 		(sheetfile "Steuereinheit.kicad_sch")
-		(attr through_hole)
+		(attr through_hole dnp)
 		(fp_line
 			(start 6.46 -1.33)
@@
 			(layers "*.Cu" "*.Mask")
 			(remove_unused_layers no)
-			(net 23 "IOB3")
+			(net 23 "EnMP")
 			(pinfunction "S")
 			(pintype "passive")
@@
 		(sheetname "/")
 		(sheetfile "Steuereinheit.kicad_sch")
-		(attr through_hole)
+		(attr through_hole dnp)
 		(fp_line
 			(start 9.12 0)
@@
 		(sheetname "/")
 		(sheetfile "Steuereinheit.kicad_sch")
-		(attr through_hole)
+		(attr through_hole dnp)
 		(fp_line
 			(start 12.44 -2.15)
@@
 		(sheetname "/")
 		(sheetfile "Steuereinheit.kicad_sch")
-		(attr through_hole)
+		(attr through_hole dnp)
 		(fp_line
 			(start 9.12 0)
@@
 		(sheetname "/")
 		(sheetfile "Steuereinheit.kicad_sch")
-		(attr through_hole)
+		(attr through_hole dnp)
 		(fp_line
 			(start 9.12 0)
@@
 		(sheetname "/")
 		(sheetfile "Steuereinheit.kicad_sch")
-		(attr through_hole)
+		(attr through_hole dnp)
 		(fp_line
 			(start -1.287288 -1.335)
@@
 		(sheetname "/")
 		(sheetfile "Steuereinheit.kicad_sch")
-		(attr through_hole)
+		(attr through_hole dnp)
 		(fp_line
 			(start 9.12 0)
@@
 		(sheetname "/")
 		(sheetfile "Steuereinheit.kicad_sch")
-		(attr through_hole)
+		(attr through_hole dnp)
 		(fp_line
 			(start -1.287288 -1.335)
