File: Serienplan/Serienplan.kicad_sch (KiCad schematic)
At the start: 73 parts, among them P1 Tasten Spalten/Zeilen 0-3, P2 Reset Serienplan, P3 Tasten Spalten/Zeilen 4-7, P7 Powernetz, P8 Zentrale, P9 Anzeigenmodule, U1 L7805, U10 74HC4094, U11 ULN2803EXT, U12 74HC107, U2 74HC245, U3 74HC165, U4 HC4051EXT, U5 TC428CPA, U6 74HC123, U7 74HC4094, U8 ULN2803EXT, U9 74HC4094

Commit message: serienplan2
Parts:
- added C30: 1nF63V, symbol Device:C
- added D12, D13, D14, D15, D16, D17: SD103C, Diode_THT:D_DO-35_SOD27_P7.62mm_Horizontal, symbol Diode:1N6857
- added R100: 47K, Resistor_THT:R_Axial_DIN0204_L3.6mm_D1.6mm_P7.62mm_Horizontal, symbol Device:R
- added R101, R94, R95, R96, R97: 2.7K, Resistor_THT:R_Axial_DIN0204_L3.6mm_D1.6mm_P7.62mm_Horizontal, symbol Device:R
- added R12: 10K, Resistor_THT:R_Axial_DIN0204_L3.6mm_D1.6mm_P7.62mm_Horizontal, symbol Device:R
Connections:
- net Anzout0: now also P9.3 (Pin_3)
- net Anzout1: now also P9.4 (Pin_4)
- net Anzout2: now also P9.5 (Pin_5)
- net Anzout3: now also P9.6 (Pin_6)
- net Anzout4: now also P9.7 (Pin_7)
- net Anzout5: now also P9.8 (Pin_8)
- net Anzout6: now also P9.9 (Pin_9)
- net Anzout7: now also P9.10 (Pin_10)
- net EnLSp: now also D13.1 (K), D14.1 (K), D15.1 (K), D16.1 (K), D17.1 (K)
- net EnLSpr: now also R12.1
- net EnLp: now also C30.1
- net EnSDAp: now also R100.2
- net GND: now also D12.2 (A), R100.1, R101.2
- net at U9.1 (STR): now also U10.1 (STR), C30.2, D12.1 (K), R101.1
- net at U9.4 (QP0): now also R97.2
- net at U9.5 (QP1): now also R96.2
- net at U9.6 (QP2): now also R95.2
- net at U9.7 (QP3): now also R94.2
- net TaktSDA: now reaches P9.11 (Pin_11), U5.7 (~{OUT_A})
- net EnSDA: now reaches P9.12 (Pin_12), U5.5 (OUT_B)
- net LS10pr: now reaches U8.5 (I5)
- net LS10pr: now also D14.2 (A), R95.1
- net LS9pr: now reaches U8.6 (I6)
- net LS9pr: now also D15.2 (A), R96.1
- net LS11pr: now reaches U8.7 (I7)
- net LS11pr: now also D16.2 (A), R94.1
- net LS8pr: now reaches U8.8 (I8)
- net LS8pr: now also D17.2 (A), R97.1
- net at U10.15 (OE): now also D13.2 (A), R12.2
Other:
- moved on the sheet: C20, D1, D2, D3, D4, D5, D6, D7, D8, P2, P7, P9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
