File: Serienplan/Serienplan.kicad_sch (KiCad schematic)
At the start: 87 parts, among them P1 Tasten Spalten/Zeilen 0-3, P2 Reset Serienplan, P3 Tasten Spalten/Zeilen 4-7, P7 Powernetz, P8 Zentrale, P9 Anzeigenmodule, U1 L7805, U10 74HC4094, U11 ULN2803EXT, U12 74HC107, U2 74HC245, U3 74HC165, U4 HC4051EXT, U5 TC428CPA, U6 74HC123, U7 74HC4094, U8 ULN2803EXT, U9 74HC4094

Commit message: size mosfet
Parts:
- added P4: Lampenzeilen, Connector_Stocko:Stocko_MKS_1666-6-0-1616_1x16_P2.50mm_Vertical, symbol Connector_Generic:Conn_01x16
- added P5: Lampenspalten, Connector_Stocko:Stocko_MKS_1662-6-0-1212_1x12_P2.50mm_Vertical, symbol Connector_Generic:Conn_01x12
- added Q1, Q10, Q13, Q17, Q18, Q2, Q5, Q9: BUZ11, Package_TO_SOT_THT:TO-220-3_Horizontal_TabUp, symbol Transistor_FET:BUZ11
- added Q11, Q12, Q14, Q15, Q16, Q19, Q20, Q3, Q4, Q6, Q7, Q8: RFP8P05, Package_TO_SOT_THT:TO-220-3_Horizontal_TabUp, symbol Transistor_FET:Q_PMOS_GDS
- P1, P7: footprint (none) -> Connector_Stocko:Stocko_MKS_1660-6-0-1010_1x10_P2.50mm_Vertical
- P2: footprint (none) -> Connector_Stocko:Stocko_MKS_1654-6-0-404_1x4_P2.50mm_Vertical
- P3, P8: footprint (none) -> Connector_Stocko:Stocko_MKS_1658-6-0-808_1x8_P2.50mm_Vertical
- P9: footprint (none) -> Connector_Stocko:Stocko_MKS_1664-6-0-1414_1x14_P2.50mm_Vertical
Connections:
- net GND: now also Q1.3 (S), Q10.3 (S), Q13.3 (S), Q17.3 (S), Q18.3 (S), Q2.3 (S), Q5.3 (S), Q9.3 (S)
- net LINE: now reaches P7.1 (Pin_1)
- net LINE: now also P2.1 (Pin_1), P7.2 (Pin_2), P7.3 (Pin_3), Q11.3 (S), Q12.3 (S), Q14.3 (S), Q15.3 (S), Q16.3 (S), Q19.3 (S), Q20.3 (S), Q3.3 (S), Q4.3 (S), Q6.3 (S), Q7.3 (S), Q8.3 (S)
- new net LS0: P5.1 (Pin_1), Q6.2 (D)
- new net LS1: P5.2 (Pin_2), Q14.2 (D)
- new net LS10: P5.11 (Pin_11), Q8.2 (D)
- new net LS11: P5.12 (Pin_12), Q16.2 (D)
- new net LS2: P5.3 (Pin_3), Q3.2 (D)
- new net LS3: P5.4 (Pin_4), Q11.2 (D)
- new net LS4: P5.5 (Pin_5), Q19.2 (D)
- new net LS5: P5.6 (Pin_6), Q7.2 (D)
- new net LS6: P5.7 (Pin_7), Q15.2 (D)
- new net LS7: P5.8 (Pin_8), Q4.2 (D)
- new net LS8: P5.9 (Pin_9), Q12.2 (D)
- new net LS9: P5.10 (Pin_10), Q20.2 (D)
- new net LZ0: P4.1 (Pin_1), P4.2 (Pin_2), Q1.2 (D)
- new net LZ1: P4.3 (Pin_3), P4.4 (Pin_4), Q9.2 (D)
- new net LZ2: P4.5 (Pin_5), P4.6 (Pin_6), Q17.2 (D)
- new net LZ3: P4.7 (Pin_7), P4.8 (Pin_8), Q5.2 (D)
- new net LZ4: P4.10 (Pin_10), P4.9 (Pin_9), Q13.2 (D)
- new net LZ5: P4.11 (Pin_11), P4.12 (Pin_12), Q2.2 (D)
- new net LZ6: P4.13 (Pin_13), P4.14 (Pin_14), Q10.2 (D)
- new net LZ7: P4.15 (Pin_15), P4.16 (Pin_16), Q18.2 (D)
Other:
- moved on the sheet: P2, P7, U12C, U6C
