File: Serienplan/Serienplan.kicad_pcb (KiCad board)
At the start: 2 copper layers, 225 x 100 mm, 63 parts, among them U1 L7805, U10 74HC4094, U11 ULN2803EXT, U12 74HC107, U2 74HC245, U3 74HC165, U4 HC4051EXT, U5 TC428CPA, U6 74HC123, U7 74HC4094, U8 ULN2803EXT, U9 74HC4094

Commit message: size mosfet
Parts:
- added D12: SD103C, Diode_THT:D_DO-35_SOD27_P7.62mm_Horizontal, F.Cu at (-37.6, -37.8)
- added D13: SD103C, Diode_THT:D_DO-35_SOD27_P7.62mm_Horizontal, F.Cu at (-37.6, -34.2)
- added D14: SD103C, Diode_THT:D_DO-35_SOD27_P7.62mm_Horizontal, F.Cu at (-37.6, -30.6)
- added D15: SD103C, Diode_THT:D_DO-35_SOD27_P7.62mm_Horizontal, F.Cu at (-37.6, -27.1)
- added D16: SD103C, Diode_THT:D_DO-35_SOD27_P7.62mm_Horizontal, F.Cu at (-37.6, -23.6)
- added D17: SD103C, Diode_THT:D_DO-35_SOD27_P7.62mm_Horizontal, F.Cu at (-37.6, -20.0)
- added P1: Tasten Spalten/Zeilen 0-3, Connector_Stocko:Stocko_MKS_1660-6-0-1010_1x10_P2.50mm_Vertical, F.Cu at (53.1, 54.0)
- added P2: Reset Serienplan, Connector_Stocko:Stocko_MKS_1654-6-0-404_1x4_P2.50mm_Vertical, F.Cu at (82.7, 54.0)
- added P3: Tasten Spalten/Zeilen 4-7, Connector_Stocko:Stocko_MKS_1658-6-0-808_1x8_P2.50mm_Vertical, F.Cu at (114.6, 54.0)
- added P4: Lampenzeilen, Connector_Stocko:Stocko_MKS_1666-6-0-1616_1x16_P2.50mm_Vertical, F.Cu at (138.4, 54.0)
- added P5: Lampenspalten, Connector_Stocko:Stocko_MKS_1662-6-0-1212_1x12_P2.50mm_Vertical, F.Cu at (203.8, 54.0)
- added P7: Powernetz, Connector_Stocko:Stocko_MKS_1660-6-0-1010_1x10_P2.50mm_Vertical, F.Cu at (46.4, 69.8)
- added P8: Zentrale, Connector_Stocko:Stocko_MKS_1658-6-0-808_1x8_P2.50mm_Vertical, F.Cu at (46.4, 94.0)
- added P9: Anzeigenmodule, Connector_Stocko:Stocko_MKS_1664-6-0-1414_1x14_P2.50mm_Vertical, F.Cu at (46.4, 134.1)
- added Q1: BUZ11, Package_TO_SOT_THT:TO-220-3_Horizontal_TabUp, F.Cu at (121.9, 72.4)
- added Q10: BUZ11, Package_TO_SOT_THT:TO-220-3_Horizontal_TabUp, F.Cu at (148.0, 94.0)
- added Q11: RFP8P05, Package_TO_SOT_THT:TO-220-3_Horizontal_TabUp, F.Cu at (190.3, 94.0)
- added Q12: RFP8P05, Package_TO_SOT_THT:TO-220-3_Horizontal_TabUp, F.Cu at (215.8, 94.0)
- added Q13: BUZ11, Package_TO_SOT_THT:TO-220-3_Horizontal_TabUp, F.Cu at (135.3, 104.8)
- added Q14: RFP8P05, Package_TO_SOT_THT:TO-220-3_Horizontal_TabUp, F.Cu at (177.0, 104.8)
- added Q15: RFP8P05, Package_TO_SOT_THT:TO-220-3_Horizontal_TabUp, F.Cu at (202.4, 104.8)
- added Q16: RFP8P05, Package_TO_SOT_THT:TO-220-3_Horizontal_TabUp, F.Cu at (245.1, 163.2)
- added Q17: BUZ11, Package_TO_SOT_THT:TO-220-3_Horizontal_TabUp, F.Cu at (121.9, 115.6)
- added Q18: BUZ11, Package_TO_SOT_THT:TO-220-3_Horizontal_TabUp, F.Cu at (148.0, 115.6)
- added Q19: RFP8P05, Package_TO_SOT_THT:TO-220-3_Horizontal_TabUp, F.Cu at (190.3, 115.6)
- added Q2: BUZ11, Package_TO_SOT_THT:TO-220-3_Horizontal_TabUp, F.Cu at (148.0, 72.4)
- added Q20: RFP8P05, Package_TO_SOT_THT:TO-220-3_Horizontal_TabUp, F.Cu at (215.8, 115.6)
- added Q3: RFP8P05, Package_TO_SOT_THT:TO-220-3_Horizontal_TabUp, F.Cu at (190.3, 72.4)
- added Q4: RFP8P05, Package_TO_SOT_THT:TO-220-3_Horizontal_TabUp, F.Cu at (215.8, 72.4)
- added Q5: BUZ11, Package_TO_SOT_THT:TO-220-3_Horizontal_TabUp, F.Cu at (135.3, 83.2)
- added Q6: RFP8P05, Package_TO_SOT_THT:TO-220-3_Horizontal_TabUp, F.Cu at (177.0, 83.2)
- added Q7: RFP8P05, Package_TO_SOT_THT:TO-220-3_Horizontal_TabUp, F.Cu at (202.4, 83.2)
- added Q8: RFP8P05, Package_TO_SOT_THT:TO-220-3_Horizontal_TabUp, F.Cu at (281.9, 123.2)
- added Q9: BUZ11, Package_TO_SOT_THT:TO-220-3_Horizontal_TabUp, F.Cu at (121.9, 94.0)
- added R100: 47K, Resistor_THT:R_Axial_DIN0204_L3.6mm_D1.6mm_P7.62mm_Horizontal, F.Cu at (-48.3, -22.2)
- added R101: 2.7K, Resistor_THT:R_Axial_DIN0204_L3.6mm_D1.6mm_P7.62mm_Horizontal, F.Cu at (-48.3, -19.1)
- added R12: 10K, Resistor_THT:R_Axial_DIN0204_L3.6mm_D1.6mm_P7.62mm_Horizontal, F.Cu at (-48.3, -38.0)
- added R94: 2.7K, Resistor_THT:R_Axial_DIN0204_L3.6mm_D1.6mm_P7.62mm_Horizontal, F.Cu at (-48.3, -34.8)
- added R95: 2.7K, Resistor_THT:R_Axial_DIN0204_L3.6mm_D1.6mm_P7.62mm_Horizontal, F.Cu at (-48.3, -31.6)
- added R96: 2.7K, Resistor_THT:R_Axial_DIN0204_L3.6mm_D1.6mm_P7.62mm_Horizontal, F.Cu at (-48.3, -28.5)
- added R97: 2.7K, Resistor_THT:R_Axial_DIN0204_L3.6mm_D1.6mm_P7.62mm_Horizontal, F.Cu at (-48.3, -25.4)
- moved D11 134.1 mm to (136.5, 21.0)
- moved D5 134.1 mm to (122.3, 21.0)
- moved D6 134.1 mm to (125.9, 21.0)
- moved D7 134.1 mm to (129.4, 21.0)
- moved D8 134.1 mm to (133.0, 21.0)
- moved R1 128.8 mm to (39.6, 203.4), turned to 90 degrees
- moved R17 128.1 mm to (74.3, 203.4), turned to 90 degrees
- moved R2 128.0 mm to (42.8, 203.4), turned to 90 degrees
- moved R11 127.3 mm to (71.1, 203.4), turned to 90 degrees
- moved R3 127.3 mm to (45.9, 203.4), turned to 90 degrees
- moved R10 126.8 mm to (68.0, 203.4), turned to 90 degrees
- moved R4 126.7 mm to (49.1, 203.4), turned to 90 degrees
- moved R9 126.4 mm to (64.8, 203.4), turned to 90 degrees
- moved R5 126.4 mm to (52.2, 203.4), turned to 90 degrees
- moved R8 126.1 mm to (61.7, 203.4), turned to 90 degrees
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Connections:
- U10 pad 1: unconnected-(U10-STR-Pad1) -> Net-(D12-K)
- U10 pad 15: unconnected-(U10-OE-Pad15) -> Net-(D13-A)
- U10 pad 8: unconnected-(U10-V_{SS}-Pad8) -> GND
- U5 pad 5: Net-(P9-Pin_12) -> EnSDA
- U5 pad 7: Net-(P9-Pin_11) -> TaktSDA
- U8 pad 5: unconnected-(U8-I5-Pad5) -> LS10pr
- U8 pad 6: unconnected-(U8-I6-Pad6) -> LS9pr
- U8 pad 7: unconnected-(U8-I7-Pad7) -> LS11pr
- U8 pad 8: unconnected-(U8-I8-Pad8) -> LS8pr
- U9 pad 1: unconnected-(U9-STR-Pad1) -> Net-(D12-K)
- U9 pad 4: unconnected-(U9-QP0-Pad4) -> Net-(U9-QP0)
- U9 pad 5: unconnected-(U9-QP1-Pad5) -> Net-(U9-QP1)
- U9 pad 6: unconnected-(U9-QP2-Pad6) -> Net-(U9-QP2)
- U9 pad 7: unconnected-(U9-QP3-Pad7) -> Net-(U9-QP3)
Other:
- board size 225 x 100 mm -> 229.9 x 102.9 mm
